File: fmcw_radar_sch/Synth.kicad_sch (KiCad schematic)
At the start: 0 parts

Commit message: board changes
board changes
Parts:
- added C11, C5: C, symbol Device:C
- added U3: ADF4372BCCZ, CC-48-4_ADI, symbol Analog Devices:ADF4372BCCZ
Connections:
- new net: C5.1, U3.44 (REFN)
- new net: C11.1, U3.43 (REFP)
- new net +3.3V: U3.39 (CE)
- new net GND: C5.2
- new net MOSI: U3.34 (SDIO)
- new net NSS: U3.33 (*CS)
- new net REFP: C11.2
- new net SCK: U3.35 (SCLK)
- new net VDDA: U3.6 (VCC_REG_OUT)
- new net VTUNE: U3.5 (VTUNE)

Commit message: CHANGES
changes
Parts:
- renumbered C5 to C35, C11 to C36, U3 to U8
Changed lines of the file:
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@@
 		(dnp no)
 		(fields_autoplaced yes)
-		(property "Reference" "C5"
+		(property "Reference" "C35"
 			(at 39.37 80.0099 0)
 			(effects
@@
 			(project "fmcw_radar_sch"
 				(path "/435eb955-ea36-4ca2-96a0-71f0d07942fb/d1630b9a-4bb5-4641-bc1b-762a2a8515ab"
-					(reference "C5")
+					(reference "C35")
 					(unit 1)
 				)
@@
 		(dnp no)
 		(fields_autoplaced yes)
-		(property "Reference" "#PWR023"
+		(property "Reference" "#PWR069"
 			(at 133.35 97.79 0)
 			(effects
@@
 			(project "fmcw_radar_sch"
 				(path "/435eb955-ea36-4ca2-96a0-71f0d07942fb/d1630b9a-4bb5-4641-bc1b-762a2a8515ab"
-					(reference "#PWR023")
+					(reference "#PWR069")
 					(unit 1)
 				)
@@
 		(dnp no)
 		(fields_autoplaced yes)
-		(property "Reference" "U3"
+		(property "Reference" "U8"
 			(at 97.79 59.69 0)
 			(effects
@@
 			(project "fmcw_radar_sch"
 				(path "/435eb955-ea36-4ca2-96a0-71f0d07942fb/d1630b9a-4bb5-4641-bc1b-762a2a8515ab"
-					(reference "U3")
+					(reference "U8")
 					(unit 1)
 				)
@@
 		(dnp no)
 		(fields_autoplaced yes)
-		(property "Reference" "#PWR020"
+		(property "Reference" "#PWR068"
 			(at 53.34 74.93 0)
 			(effects
@@
 			(project "fmcw_radar_sch"
 				(path "/435eb955-ea36-4ca2-96a0-71f0d07942fb/d1630b9a-4bb5-4641-bc1b-762a2a8515ab"
-					(reference "#PWR020")
+					(reference "#PWR068")
 					(unit 1)
 				)
@@
 		(dnp no)
 		(fields_autoplaced yes)
-		(property "Reference" "#PWR019"
+		(property "Reference" "#PWR067"
 			(at 35.56 93.98 0)
 			(effects
@@
 			(project "fmcw_radar_sch"
 				(path "/435eb955-ea36-4ca2-96a0-71f0d07942fb/d1630b9a-4bb5-4641-bc1b-762a2a8515ab"
-					(reference "#PWR019")
+					(reference "#PWR067")
 					(unit 1)
 				)
@@
 		(dnp no)
 		(fields_autoplaced yes)
-		(property "Reference" "C11"
+		(property "Reference" "C36"
 			(at 49.53 80.0099 0)
 			(effects
@@
 			(project "fmcw_radar_sch"
 				(path "/435eb955-ea36-4ca2-96a0-71f0d07942fb/d1630b9a-4bb5-4641-bc1b-762a2a8515ab"
-					(reference "C11")
-					(unit 1)
-				)
+					(reference "C36")
+					(unit 1)
+				)
