File: fmcw_radar_sch/fmcw_radar_sch.kicad_pcb (KiCad board)
At the start: 4 copper layers, 100 x 100 mm, 93 parts, among them J1 2x5 1.27mm, J10 Screw_Terminal_01x05, J11 Conn_Coaxial, J2 Conn_01x04_Pin, J3 Conn_01x07_Pin, J4 Conn_01x05_Pin, J5 Conn_01x04_Pin, J6 Conn_01x03_Pin, J7 Conn_01x04_Pin, J8 USB_C_Receptacle_USB2.0_16P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

Commit message: Update fmcw_radar_sch.kicad_pcb
Parts:
- added ?: , , F.Cu at (145.3, 58.8)
- added ?: , , F.Cu at (150.1, 58.1)
- added ?: , , F.Cu at (150.1, 58.8)
- added ?: , , F.Cu at (143.0, 58.1)
- added ?: , , F.Cu at (145.3, 58.1)
- added ?: , , F.Cu at (147.7, 58.8)
- added ?: , , F.Cu at (143.0, 58.8)
- added ?: , , F.Cu at (147.7, 58.1)
- added CR2: ESD701DPYRQ1, nonkicad:X1SON2_DPY_TEX, F.Cu at (191.8, 110.6)
- added CR2: ESD701DPYRQ1, nonkicad:X1SON2_DPY_TEX, F.Cu at (140.3, 143.5)
- added CR2: ESD701DPYRQ1, nonkicad:X1SON2_DPY_TEX, F.Cu at (153.7, 143.5)
- added CR2: ESD701DPYRQ1, nonkicad:X1SON2_DPY_TEX, F.Cu at (137.7, 143.5)
- added CR2: ESD701DPYRQ1, nonkicad:X1SON2_DPY_TEX, F.Cu at (121.8, 143.7)
- added CR2: ESD701DPYRQ1, nonkicad:X1SON2_DPY_TEX, F.Cu at (152.6, 58.4)
- added CR2: ESD701DPYRQ1, nonkicad:X1SON2_DPY_TEX, F.Cu at (193.6, 83.5)
- added CR2: ESD701DPYRQ1, nonkicad:X1SON2_DPY_TEX, F.Cu at (151.1, 143.5)
- added CR2: ESD701DPYRQ1, nonkicad:X1SON2_DPY_TEX, F.Cu at (191.8, 113.2)
- added CR2: ESD701DPYRQ1, nonkicad:X1SON2_DPY_TEX, F.Cu at (119.2, 143.7)
- added CR3: ESD701DPYRQ1, nonkicad:X1SON2_DPY_TEX, F.Cu at (148.7, 143.5)
- added CR3: ESD701DPYRQ1, nonkicad:X1SON2_DPY_TEX, F.Cu at (116.8, 143.7)
- added CR3: ESD701DPYRQ1, nonkicad:X1SON2_DPY_TEX, F.Cu at (155.4, 58.4)
- added CR3: ESD701DPYRQ1, nonkicad:X1SON2_DPY_TEX, F.Cu at (191.8, 115.6)
- added CR3: ESD701DPYRQ1, nonkicad:X1SON2_DPY_TEX, F.Cu at (193.6, 85.9)
- added CR3: ESD701DPYRQ1, nonkicad:X1SON2_DPY_TEX, F.Cu at (135.3, 143.5)
- added CR4: ESD701DPYRQ1, nonkicad:X1SON2_DPY_TEX, F.Cu at (193.6, 88.3)
- added CR4: ESD701DPYRQ1, nonkicad:X1SON2_DPY_TEX, F.Cu at (132.9, 143.5)
- added CR4: ESD701DPYRQ1, nonkicad:X1SON2_DPY_TEX, F.Cu at (191.8, 117.9)
- added CR4: ESD701DPYRQ1, nonkicad:X1SON2_DPY_TEX, F.Cu at (146.3, 143.5)
- added CR4: ESD701DPYRQ1, nonkicad:X1SON2_DPY_TEX, F.Cu at (129.9, 143.8)
- added CR4: ESD701DPYRQ1, nonkicad:X1SON2_DPY_TEX, F.Cu at (110.5, 67.5)
- added CR4: ESD701DPYRQ1, nonkicad:X1SON2_DPY_TEX, F.Cu at (114.4, 143.7)
- added CR4: ESD701DPYRQ1, nonkicad:X1SON2_DPY_TEX, F.Cu at (157.7, 58.4)
- moved U3 3.03 mm to (173.3, 99.1)

Commit message: CHANGES
changes
Parts:
- added D1: ESD131-B1-W0201, Diode_SMD:Nexperia_DSN0603-2_0.6x0.3mm_P0.4mm, F.Cu at (0.62, 4.26)
- added D4: ESD131-B1-W0201, Diode_SMD:Infineon_SG-WLL-2-3_0.58x0.28_P0.36mm, F.Cu at (0.61, 0.47)
Connections:
- net Net-(U5-BST) renamed /Power System/BST
Routing:
- added copper zone on F.Cu, net /Power System/BST

Commit message: Routing
Routing
Parts:
- removed ? (x8): , 
- removed the CR2 at (191.8, 110.6)
- removed the CR2 at (140.3, 143.5)
- removed the CR2 at (153.7, 143.5)
- removed the CR2 at (137.7, 143.5)
- removed the CR2 at (121.8, 143.7)
- removed the CR2 at (152.6, 58.4)
- removed the CR2 at (193.6, 83.5)
- removed the CR2 at (151.1, 143.5)
- removed the CR2 at (191.8, 113.2)
- removed the CR2 at (119.2, 143.7)
- removed CR201: ESD701DPYRQ1, nonkicad:X1SON2_DPY_TEX
- removed the CR3 at (148.7, 143.5)
- removed the CR3 at (116.8, 143.7)
- removed the CR3 at (155.4, 58.4)
- removed the CR3 at (191.8, 115.6)
- removed the CR3 at (193.6, 85.9)
- removed the CR3 at (135.3, 143.5)
- removed the CR4 at (193.6, 88.3)
- removed the CR4 at (132.9, 143.5)
- removed the CR4 at (191.8, 117.9)
- removed the CR4 at (146.3, 143.5)
- removed the CR4 at (129.9, 143.8)
- removed the CR4 at (110.5, 67.5)
- removed the CR4 at (114.4, 143.7)
- removed the CR4 at (157.7, 58.4)
- removed D1: ESD131-B1-W0201, Diode_SMD:Nexperia_DSN0603-2_0.6x0.3mm_P0.4mm
- removed D4: ESD131-B1-W0201, Diode_SMD:Infineon_SG-WLL-2-3_0.58x0.28_P0.36mm
- moved R4 35.2 mm to (184.4, 75.1)
- moved R6 33.6 mm to (184.4, 78.7)
- moved C6 33.2 mm to (184.3, 80.8)
- moved R3 33.1 mm to (184.3, 73.3)
- moved R7 30.4 mm to (189.5, 119.7), turned to 90 degrees
- moved R5 29.7 mm to (184.3, 76.7)
- moved R19 14.3 mm to (169.2, 129.5)
- moved C39 13.8 mm to (163.9, 131.4), turned to -90 degrees
- moved R20 13.2 mm to (159.6, 125.7), turned to 90 degrees
- moved J11 13.2 mm to (181.6, 140.3)
- moved C37 13.0 mm to (167.9, 125.4)
- moved C38 13.0 mm to (168.1, 127.1)
- moved C40 13.0 mm to (170.5, 124.5)
- moved C42 13.0 mm to (178.6, 125.2)
- moved R24 13.0 mm to (181.5, 126.1)
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Connections:
- net Net-(SW2-B) renamed /Power System/V_PREfilt
- net Net-(U5-SW) renamed /Power System/SW
- R19 pad 1: SPI2_SCK -> SCK2
- U9 pad 6: SPI2_NSS -> NSS2
- U9 pad 8: SPI2_MOSI -> MOSI2
Routing:
- net +3.3VA: track 0.00 -> 161.3 mm, vias 0 -> 5
- net VBUS: track 0.00 -> 143.6 mm, vias 0 -> 3
- net MOSI2: track 0.00 -> 96.5 mm
- net NSS2: track 0.00 -> 92.8 mm, vias 0 -> 1
- net GND: track 0.00 -> 92.5 mm, vias 0 -> 36
- net SCK2: track 0.00 -> 89.4 mm, vias 0 -> 1
- net Net-(J4-Pin_2): track 0.00 -> 59.0 mm, vias 0 -> 2
- net Net-(J5-Pin_4): track 0.00 -> 59.0 mm
- net Net-(J4-Pin_1): track 0.00 -> 58.8 mm, vias 0 -> 1
- net Net-(J5-Pin_3): track 0.00 -> 57.1 mm
- net Net-(J5-Pin_2): track 0.00 -> 56.7 mm, vias 0 -> 4
- net Net-(J4-Pin_3): track 0.00 -> 55.3 mm, vias 0 -> 1
- net +3.3V: track 0.00 -> 54.8 mm, vias 0 -> 16
- net Net-(J3-Pin_7): track 0.00 -> 54.5 mm, vias 0 -> 1
- net Net-(J5-Pin_1): track 0.00 -> 53.2 mm, vias 0 -> 2
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- added copper zone on F.Cu, net +3.3VA
- added copper zone on F.Cu, net /Power System/5_volt_filt
- added copper zone on F.Cu, net /Power System/SW
- added copper zone on F.Cu, net /Power System/V_PREfilt
- removed copper zone on F.Cu, net (none)
