File: fmcw_radar_sch/fmcw_radar_sch.kicad_pcb (KiCad board)
At the start: 4 copper layers, 100 x 100 mm, 92 parts, among them J1 2x5 1.27mm, J10 Screw_Terminal_01x05, J11 Conn_Coaxial, J2 Conn_01x04_Pin, J3 Conn_01x07_Pin, J4 Conn_01x05_Pin, J5 Conn_01x04_Pin, J6 Conn_01x03_Pin, J7 Conn_01x04_Pin, J8 USB_C_Receptacle_USB2.0_16P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

Commit message: changes
changes
Routing:
- net GND: vias 36 -> 42
Changed lines of the file:
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@@
 		(tags "resistor")
 		(property "Reference" "R19"
-			(at -3.202 -0.303 0)
+			(at -0.1 -2 0)
 			(layer "F.SilkS")
 			(effects
@@
 		(tags "resistor")
 		(property "Reference" "R20"
-			(at 3.039999 0.016 90)
+			(at 2.3 0.1 180)
 			(layer "F.SilkS")
 			(effects
@@
 		(tags "capacitor")
 		(property "Reference" "C39"
-			(at 1.744 1.529 90)
+			(at 2.5 0 180)
 			(layer "F.SilkS")
 			(effects
@@
 		(tags "SOT TO_SOT_SMD")
 		(property "Reference" "U10"
-			(at 0.028 -2.6475 0)
+			(at 0.028 -3.3185 0)
 			(layer "F.SilkS")
 			(effects
@@
 	)
 	(via
+		(at 126.5015 60.82)
+		(size 0.6)
+		(drill 0.3)
+		(layers "F.Cu" "B.Cu")
+		(net 1)
+	)
+	(via
+		(at 128 61.1)
+		(size 0.6)
+		(drill 0.3)
+		(layers "F.Cu" "B.Cu")
+		(free yes)
+		(net 1)
+	)
+	(via
 		(at 176.8 122.8)
 		(size 0.6)
@@
 	)
 	(via
+		(at 126.3445 64.275)
+		(size 0.6)
+		(drill 0.3)
+		(layers "F.Cu" "B.Cu")
+		(net 1)
+	)
+	(via
 		(at 138.7 86.3)
 		(size 0.6)
@@
 	)
 	(via
+		(at 127.9 62.9)
+		(size 0.6)
+		(drill 0.3)
+		(layers "F.Cu" "B.Cu")
+		(free yes)
+		(net 1)
+	)
+	(via
 		(at 153.7 63.3)
 		(size 0.6)
@@
 	)
 	(via
+		(at 127.9 65.3)
+		(size 0.6)
+		(drill 0.3)
+		(layers "F.Cu" "B.Cu")
+		(free yes)
+		(net 1)
+	)
+	(via
 		(at 152.3 98)
 		(size 0.6)
@@
 	)
 	(via
+		(at 127.9 64.2)
+		(size 0.6)
+		(drill 0.3)
+		(layers "F.Cu" "B.Cu")
+		(free yes)
+		(net 1)
+	)
+	(via
 		(at 150.9 63.2)
 		(size 0.6)
@@
 	)
 	(via
-		(at 124.5 67.4)
+		(at 124.6 67.8)
 		(size 0.6)
 		(drill 0.3)
@@
 	)
 	(via
-		(at 124.5 69)
+		(at 124.6 69)
 		(size 0.6)
 		(drill 0.3)

Commit message: a lot of updates
usb power delivery + finishing touches
Routing:
- net /Power System/5_volt_filt: vias 9 -> 0
Changed lines of the file:
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@@
-		(net 5)
-	)
-	(via
-		(at 130.95 83)
-		(size 0.6)
-		(drill 0.3)
-		(layers "F.Cu" "B.Cu")
-		(free yes)
-		(net 5)
-	)
-	(via
-		(at 132.7625 83)
-		(size 0.6)
-		(drill 0.3)
-		(layers "F.Cu" "B.Cu")
-		(free yes)
-		(net 5)
-	)
-	(via
-		(at 136.3875 83)
-		(size 0.6)
-		(drill 0.3)
-		(layers "F.Cu" "B.Cu")
-		(free yes)
-		(net 5)
-	)
-	(via
-		(at 129.1375 83)
-		(size 0.6)
-		(drill 0.3)
-		(layers "F.Cu" "B.Cu")
-		(free yes)
-		(net 5)
-	)
-	(via
-		(at 134.575 83)
-		(size 0.6)
-		(drill 0.3)
-		(layers "F.Cu" "B.Cu")
-		(free yes)
-		(net 5)
-	)
-	(via
-		(at 125.5125 83)
-		(size 0.6)
-		(drill 0.3)
-		(layers "F.Cu" "B.Cu")
-		(free yes)
-		(net 5)
-	)
-	(via
-		(at 138.2 83)
-		(size 0.6)
-		(drill 0.3)
-		(layers "F.Cu" "B.Cu")
-		(free yes)
-		(net 5)
-	)
-	(via
-		(at 123.7 83)
-		(size 0.6)
-		(drill 0.3)
-		(layers "F.Cu" "B.Cu")
-		(free yes)
-		(net 5)
-	)
-	(via
-		(at 127.325 83)
-		(size 0.6)
-		(drill 0.3)
-		(layers "F.Cu" "B.Cu")
-		(free yes)
 		(net 5)
 	)

Commit message: Silkscreen finishing
Silkscreen finishting
Other:
- board text added: "+1V8 +2V5 +3.3VA +3.3V +5V"
- board text added: "+BAT"
- board text added: "BATT USB"
- board text added: "BOOT0"
- board text added: "MOSI2 MISO2 SCK2 NSS2"
- board text added: "NSS SCK MISO MOSI"
- board text added: "PA 0 1 2 3 4"
- board text added: "PA8 9 10"
- board text added: "PB 11 9 8 7 6 5 4"
- board text added: "PC 13 14 15 PB0 PB1"
- board text added: "SWD"
- board text added: "VCO Tune"
Changed lines of the file:
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@@
 			(at 0 -2.38 90)
 			(layer "F.SilkS")
+			(hide yes)
 			(effects
 				(font
@@
 			(at 3.99 -2.99 0)
 			(layer "F.SilkS")
+			(hide yes)
 			(effects
 				(font
@@
 			(at 0.297 -7.239 180)
 			(layer "F.SilkS")
+			(hide yes)
 			(effects
 				(font
@@
 			(at 0 -2.38 90)
 			(layer "F.SilkS")
+			(hide yes)
 			(effects
 				(font
@@
 			(at 0 -2.38 0)
 			(layer "F.SilkS")
+			(hide yes)
 			(effects
 				(font
@@
 			(at 0 -2.38 90)
 			(layer "F.SilkS")
+			(hide yes)
 			(effects
 				(font
@@
 			(at 0 -2.9 0)
 			(layer "F.SilkS")
+			(hide yes)
 			(effects
 				(font
@@
 			(at -2.425 0.3 180)
 			(layer "F.SilkS")
+			(hide yes)
 			(effects
 				(font
@@
 			(at -3.813 -0.07 0)
 			(layer "F.SilkS")
+			(hide yes)
 			(effects
 				(font
@@
 			(at -3.698 -0.082 0)
 			(layer "F.SilkS")
+			(hide yes)
 			(effects
 				(font
@@
 			(at 3.99 -2.99 0)
 			(layer "F.SilkS")
+			(hide yes)
 			(effects
 				(font
@@
 			(at -0.249 -2.219 0)
 			(layer "F.SilkS")
+			(hide yes)
 			(effects
 				(font
@@
 		(layer "Edge.Cuts")
 	)
+	(gr_text "VCO Tune\n"
+		(at 162.21 147.56 0)
+		(layer "F.SilkS" knockout)
+		(effects
+			(font
+				(size 1.5 1.5)
+				(thickness 0.3)
+				(bold yes)
+				(italic yes)
+			)
+			(justify left bottom)
+		)
+	)
+	(gr_text "PC 13 14 15 PB0 PB1"
+		(at 124.37 144.57 0)
+		(layer "F.SilkS" knockout)
+		(effects
+			(font
+				(size 1 1)
+				(thickness 0.2)
+				(bold yes)
+				(italic yes)
+			)
+			(justify left bottom)
+		)
+	)
+	(gr_text "PA8 9 10\n"
+		(at 194.48 89.55 90)
+		(layer "F.SilkS" knockout)
+		(effects
+			(font
+				(size 1 1)
+				(thickness 0.2)
+				(bold yes)
+				(italic yes)
+			)
+			(justify left bottom)
+		)
+	)
+	(gr_text "+BAT"
+		(at 101.23 76.39 0)
+		(layer "F.SilkS" knockout)
+		(effects
+			(font
+				(size 1.5 1.5)
+				(thickness 0.3)
+				(bold yes)
+				(italic yes)
+			)
+			(justify left bottom)
+		)
+	)
+	(gr_text "NSS SCK MISO MOSI"
+		(at 142.07 144.54 0)
+		(layer "F.SilkS" knockout)
+		(effects
+			(font
+				(size 1 1)
+				(thickness 0.25)
+				(bold yes)
+				(italic yes)
+			)
+			(justify left bottom)
+		)
+	)
+	(gr_text "+1V8 +2V5 +3.3VA +3.3V +5V"
+		(at 163.15 64.36 0)
+		(layer "F.SilkS" knockout)
+		(effects
+			(font
+				(size 1 1)
+				(thickness 0.2)
+				(bold yes)
+				(italic yes)
+			)
+			(justify left bottom)
+		)
+	)
+	(gr_text "BATT USB"
+		(at 111.51 58.86 0)
+		(layer "F.SilkS" knockout)
+		(effects
+			(font
+				(size 1.5 1.5)
+				(thickness 0.25)
+				(bold yes)
+				(italic yes)
+			)
+			(justify left bottom)
+		)
+	)
+	(gr_text "MOSI2 MISO2 SCK2 NSS2"
+		(at 192.61 106.28 270)
+		(layer "F.SilkS" knockout)
+		(effects
+			(font
+				(size 1 1)
+				(thickness 0.2)
+				(bold yes)
+				(italic yes)
+			)
+			(justify left bottom)
+		)
+	)
+	(gr_text "SWD"
+		(at 195.46 64.2 0)
+		(layer "F.SilkS" knockout)
+		(effects
+			(font
+				(size 1 1)
+				(thickness 0.2)
+				(bold yes)
+				(italic yes)
+			)
+			(justify left bottom)
+		)
+	)
+	(gr_text "BOOT0"
+		(at 123.11 58.86 0)
+		(layer "F.SilkS" knockout)
+		(effects
+			(font
+				(size 1.5 1.5)
+				(thickness 0.3)
+				(bold yes)
+				(italic yes)
+			)
+			(justify left bottom)
+		)
+	)
+	(gr_text "PA 0 1 2 3 4"
+		(at 111.74 145.21 0)
+		(layer "F.SilkS" knockout)
+		(effects
+			(font
+				(size 1 1)
+				(thickness 0.2)
+				(bold yes)
+				(italic yes)
+			)
+			(justify left bottom)
+		)
+	)
+	(gr_text "PB 11 9 8 7 6 5 4 "
+		(at 136.63 58.24 0)
+		(layer "F.SilkS" knockout)
+		(effects
+			(font
+				(size 1.5 1.5)
+				(thickness 0.25)
+				(bold yes)
+				(italic yes)
+			)
+			(justify left bottom)
+		)
+	)
 	(segment

Commit message: changes from yesterday
changes from yesterday
Routing:
- net Net-(J3-Pin_1): vias 1 -> 2
- net GND: vias 42 -> 54
Changed lines of the file:
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@@
 	)
 	(via
+		(at 151 77)
+		(size 0.6)
+		(drill 0.3)
+		(layers "F.Cu" "B.Cu")
+		(free yes)
+		(net 1)
+	)
+	(via
 		(at 180.2 125.6)
 		(size 0.6)
@@
 	)
 	(via
+		(at 152 81)
+		(size 0.6)
+		(drill 0.3)
+		(layers "F.Cu" "B.Cu")
+		(free yes)
+		(net 1)
+	)
+	(via
 		(at 169.5 127.6)
 		(size 0.6)
@@
 	)
 	(via
+		(at 153 77)
+		(size 0.6)
+		(drill 0.3)
+		(layers "F.Cu" "B.Cu")
+		(free yes)
+		(net 1)
+	)
+	(via
+		(at 154 79)
+		(size 0.6)
+		(drill 0.3)
+		(layers "F.Cu" "B.Cu")
+		(free yes)
+		(net 1)
+	)
+	(via
 		(at 176.6 99.3)
 		(size 0.6)
@@
 	)
 	(via
+		(at 154 78)
+		(size 0.6)
+		(drill 0.3)
+		(layers "F.Cu" "B.Cu")
+		(free yes)
+		(net 1)
+	)
+	(via
+		(at 154 77)
+		(size 0.6)
+		(drill 0.3)
+		(layers "F.Cu" "B.Cu")
+		(free yes)
+		(net 1)
+	)
+	(via
 		(at 162.6 85.1)
 		(size 0.6)
@@
 	)
 	(via
+		(at 151.356001 79.296401)
+		(size 0.6)
+		(drill 0.3)
+		(layers "F.Cu" "B.Cu")
+		(net 1)
+	)
+	(via
 		(at 153.8 81)
 		(size 0.6)
@@
 	)
 	(via
+		(at 154 83)
+		(size 0.6)
+		(drill 0.3)
+		(layers "F.Cu" "B.Cu")
+		(free yes)
+		(net 1)
+	)
+	(via
+		(at 154 80)
+		(size 0.6)
+		(drill 0.3)
+		(layers "F.Cu" "B.Cu")
+		(free yes)
+		(net 1)
+	)
+	(via
+		(at 151 81)
+		(size 0.6)
+		(drill 0.3)
+		(layers "F.Cu" "B.Cu")
+		(free yes)
+		(net 1)
+	)
+	(via
 		(at 189.9 103.5)
 		(size 0.6)
@@
 	)
 	(via
+		(at 154 82)
+		(size 0.6)
+		(drill 0.3)
+		(layers "F.Cu" "B.Cu")
+		(free yes)
+		(net 1)
+	)
+	(via
 		(at 127.2 102.5)
 		(size 0.6)
@@
 	)
 	(via
+		(at 152 77)
+		(size 0.6)
+		(drill 0.3)
+		(layers "F.Cu" "B.Cu")
+		(free yes)
+		(net 1)
+	)
+	(via
 		(at 150.9 63.2)
 		(size 0.6)
@@
 		(start 191.214 99.447)
 		(end 192.086 99.447)
-		(width 0.2)
+		(width 0.155)
 		(layer "F.Cu")
 		(net 20)
@@
 		(start 192.086 100.447)
 		(end 191.214 100.447)
-		(width 0.2)
+		(width 0.155)
 		(layer "F.Cu")
 		(net 20)
@@
 		(start 175.947 100.447)
 		(end 191.214 100.447)
-		(width 0.25)
+		(width 0.155)
 		(layer "F.Cu")
 		(net 20)
 	)
 	(segment
-		(start 192.086 99.447)
-		(end 192.135 99.496)
-		(width 0.2)
+		(start 174.622 100.0295)
+		(end 175.5295 100.0295)
+		(width 0.155)
 		(layer "F.Cu")
 		(net 20)
 	)
 	(segment
-		(start 192.135 100.398)
-		(end 192.086 100.447)
-		(width 0.2)
+		(start 192.135 99.496)
+		(end 192.086 99.447)
+		(width 0.155)
 		(layer "F.Cu")
 		(net 20)
 	)
 	(segment
-		(start 174.622 100.0295)
-		(end 175.5295 100.0295)
-		(width 0.25)
+		(start 175.5295 100.0295)
+		(end 175.947 100.447)
+		(width 0.155)
 		(layer "F.Cu")
 		(net 20)
 	)
 	(segment
-		(start 175.5295 100.0295)
-		(end 175.947 100.447)
-		(width 0.25)
+		(start 192.086 100.447)
+		(end 192.135 100.398)
+		(width 0.155)
 		(layer "F.Cu")
 		(net 20)
@@
 		(start 192.135 99.496)
 		(end 192.135 100.398)
-		(width 0.2)
+		(width 0.155)
 		(layer "F.Cu")
 		(net 20)
@@
 		(start 175.8705 98.1295)
 		(end 176.2 97.8)
-		(width 0.25)
+		(width 0.155)
 		(layer "F.Cu")
 		(net 21)
@@
 		(start 190.293 99.898)
 		(end 190.293 99.054)
-		(width 0.2)
+		(width 0.155)
 		(layer "F.Cu")
 		(net 21)
@@
 		(start 191.214 98.947)
 		(end 190.4 98.947)
-		(width 0.2)
+		(width 0.155)
 		(layer "F.Cu")
 		(net 21)
@@
 		(start 174.622 98.1295)
 		(end 175.8705 98.1295)
-		(width 0.25)
+		(width 0.155)
+		(layer "F.Cu")
+		(net 21)
+	)
+	(segment
+		(start 190.293 99.898)
+		(end 190.342 99.947)
+		(width 0.155)
 		(layer "F.Cu")
 		(net 21)
@@
 		(start 188.947 98.947)
 		(end 190.4 98.947)
-		(width 0.25)
+		(width 0.155)
 		(layer "F.Cu")
 		(net 21)
@@
 		(start 176.2 97.8)
 		(end 187.8 97.8)
-		(width 0.25)
+		(width 0.155)
 		(layer "F.Cu")
 		(net 21)
 	)
 	(segment
-		(start 190.342 99.947)
-		(end 190.293 99.898)
-		(width 0.2)
+		(start 191.214 99.947)
+		(end 190.342 99.947)
+		(width 0.155)
 		(layer "F.Cu")
 		(net 21)
@@
 		(start 190.293 99.054)
 		(end 190.4 98.947)
-		(width 0.2)
-		(layer "F.Cu")
-		(net 21)
-	)
-	(segment
-		(start 191.214 99.947)
-		(end 190.342 99.947)
-		(width 0.2)
+		(width 0.155)
 		(layer "F.Cu")
 		(net 21)
@@
 		(start 187.8 97.8)
 		(end 188.947 98.947)
-		(width 0.25)
+		(width 0.155)
 		(layer "F.Cu")
 		(net 21)
@@
 		(start 155.293751 98.775)
 		(end 170.106499 98.775)
-		(width 0.2)
+		(width 0.155)
 		(layer "F.Cu")
 		(net 41)
@@
 		(start 170.751999 98.1295)
 		(end 171.922 98.1295)
-		(width 0.2)
+		(width 0.155)
 		(layer "F.Cu")
 		(net 41)
@@
 		(start 170.106499 98.775)
 		(end 170.751999 98.1295)
-		(width 0.2)
+		(width 0.155)
 		(layer "F.Cu")
 		(net 41)
@@
 		(start 154.1625 98.75)
 		(end 155.268751 98.75)
-		(width 0.2)
+		(width 0.155)
 		(layer "F.Cu")
 		(net 41)
 	)
 	(segment
-		(start 155.268751 99.25)
-		(end 155.293751 99.225)
-		(width 0.2)
-		(layer "F.Cu")
-		(net 42)
-	)
-	(segment
 		(start 155.293751 99.225)
 		(end 169.947499 99.225)
-		(width 0.2)
+		(width 0.155)
 		(layer "F.Cu")
 		(net 42)
@@
 		(start 170.751999 100.0295)
 		(end 171.922 100.0295)
-		(width 0.2)
+		(width 0.155)
 		(layer "F.Cu")
 		(net 42)
@@
 		(start 169.947499 99.225)
 		(end 170.751999 100.0295)
-		(width 0.2)
+		(width 0.155)
 		(layer "F.Cu")
 		(net 42)
@@
 		(start 154.1625 99.25)
 		(end 155.268751 99.25)
-		(width 0.2)
+		(width 0.155)
 		(layer "F.Cu")
 		(net 42)
@@
 		(net 58)
 	)
+	(via
+		(at 149.9 77)
+		(size 0.6)
+		(drill 0.3)
+		(layers "F.Cu" "B.Cu")
+		(net 58)
+	)
 	(segment
-		(start 149.9 59.9)
+		(start 149.9 77)
 		(end 149.9 81.6)
 		(width 0.3)
 		(layer "B.Cu")
+		(net 58)
+	)
+	(segment
+		(start 149.9 59.9)
+		(end 149.9 77)
+		(width 0.3)
+		(layer "B.Cu")
