File: fmcw_radar_sch/Up_Down_Converter/Up_Down_Converter.kicad_pcb (KiCad board)
At the start: 4 copper layers, 100 x 100 mm, 80 parts, among them J1 Conn_01x04_Pin, J10 Screw_Terminal_01x05, J14 Conn_01x05_Pin, J15 RJ45, J2 Conn_01x04_Pin, J3 Conn_Coaxial, J4 Conn_01x04_Pin, J5 Conn_01x05_Pin, J7 Conn_01x01_Pin, J8 USB_C_Receptacle_USB2.0_16P, J9 Screw_Terminal_01x02, SW1 SW_Nidec_CAS-120A1, U1 ADAR2004ACCZ, U2 LP3875EMP-2.5/NOPB, U3 USBLC6-2SC6, U4 TLV75718PDYDR, U5 AP63203WU, U6 HT7533-1, U7 ADAR2001ACCZ, U9 ADF4372BCCZ

Commit message: initial
initial
Parts:
- removed J10: Screw_Terminal_01x05, TerminalBlock_Phoenix:TerminalBlock_Phoenix_MKDS-3-5-5.08_1x05_P5.08mm_Horizontal
- moved D5 117.4 mm to (164.0, 144.4), turned to 180 degrees
- moved C18 117.1 mm to (160.4, 144.3), turned to 180 degrees
- moved R1 115.6 mm to (152.1, 143.0), turned to -90 degrees
- moved C15 114.8 mm to (157.9, 140.9), turned to -90 degrees
- moved R15 114.7 mm to (167.7, 144.4)
- moved C19 84.5 mm to (134.4, 126.5), turned to -90 degrees
- moved C21 83.0 mm to (132.0, 132.7), turned to -90 degrees
- moved C17 78.9 mm to (125.0, 126.2), turned to -90 degrees
- moved C24 77.4 mm to (124.6, 135.2), turned to 180 degrees
- moved C12 73.9 mm to (111.0, 130.8), turned to 180 degrees
- moved D7 72.7 mm to (122.3, 133.3)
- moved D3 69.0 mm to (111.7, 137.1)
- moved L2 68.0 mm to (130.1, 125.6)
- moved R17 66.5 mm to (122.9, 130.2), turned to 90 degrees
- moved R14 65.6 mm to (109.1, 136.1), turned to 90 degrees
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Routing:
- net MOSI: track 0.00 -> 100.7 mm, vias 0 -> 8
- net SCK: track 0.00 -> 98.6 mm, vias 0 -> 5
- net +3.3V: track 13.6 -> 98.2 mm, vias 0 -> 2
- net IFOUT3+: track 0.00 -> 76.9 mm, vias 0 -> 4
- net IFOUT3-: track 0.00 -> 74.1 mm, vias 0 -> 4
- net IFOUT4+: track 0.00 -> 72.2 mm, vias 0 -> 2
- net IFOUT1+: track 0.00 -> 69.5 mm, vias 0 -> 1
- net IFOUT4-: track 0.00 -> 69.1 mm, vias 0 -> 2
- net IFOUT2+: track 0.00 -> 67.8 mm, vias 0 -> 2
- net +1V8: track 8.56 -> 76.0 mm, vias 0 -> 2
- net IFOUT1-: track 0.00 -> 66.2 mm, vias 0 -> 1
- net IFOUT2-: track 0.00 -> 64.6 mm, vias 0 -> 2
- net MISO: track 0.00 -> 64.0 mm, vias 0 -> 5
- net VCC: track 0.00 -> 54.5 mm, vias 0 -> 6
- net +5V: track 0.00 -> 53.7 mm, vias 0 -> 2
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- added copper zone on F.Cu, net +5V
- added copper zone on F.Cu, net VPOS4R

Commit message: a lot of updates
usb power delivery + finishing touches
Parts:
- removed J1: Conn_01x04_Pin, Connector_PinHeader_2.54mm:PinHeader_1x04_P2.54mm_Vertical
- removed J14, J5: Conn_01x05_Pin, Connector_PinHeader_2.54mm:PinHeader_1x05_P2.54mm_Vertical
- removed J7: Conn_01x01_Pin, Connector_PinHeader_2.54mm:PinHeader_1x01_P2.54mm_Vertical
- removed J9: Screw_Terminal_01x02, TerminalBlock:TerminalBlock_MaiXu_MX126-5.0-02P_1x02_P5.00mm
- moved R9 270.4 mm to (376.3, 64.1), turned to 0 degrees
- moved R13 270.1 mm to (376.3, 67.4)
- moved R14 269.7 mm to (363.9, 47.6), turned to 0 degrees
- moved U3 264.9 mm to (375.0, 72.6), turned to 0 degrees
- moved R10 263.8 mm to (359.5, 52.6), turned to 0 degrees
- moved U2 257.4 mm to (368.8, 73.3)
- moved C14 254.9 mm to (350.8, 50.1), turned to 0 degrees
- moved C12 254.7 mm to (350.8, 45.1), turned to 0 degrees
- moved R12 253.0 mm to (363.9, 45.1), turned to 0 degrees
- moved U6 252.7 mm to (369.9, 59.5)
- moved R17 252.4 mm to (363.9, 55.1), turned to 0 degrees
- moved J8 251.9 mm to (358.9, 71.8)
- moved R11 251.6 mm to (359.5, 55.1), turned to 0 degrees
- moved J3 251.4 mm to (353.2, 83.1)
- moved D4 251.2 mm to (372.3, 52.3), turned to 0 degrees
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Connections:
- C2 pad 2: Net-(U9-REFP) -> unconnected-(C2-Pad2)
- U7 pad 18: RF4O+ -> GND
- U7 pad 19: RF4O- -> GND
- U7 pad 23: RFO3+ -> GND
- U7 pad 24: RFO3- -> GND
- U7 pad 28: RFO2- -> GND
- U7 pad 29: RFO2+ -> GND
- U7 pad 33: RFO1- -> GND
- U7 pad 34: RFO1+ -> GND
Routing:
- net GND: track 46.4 -> 235.3 mm, vias 1024 -> 620
- net +3.3V: track 98.2 -> 0.00 mm, vias 2 -> 0
- net IFOUT3+: track 76.9 -> 2.26 mm, vias 4 -> 0
- net MOSI: track 100.7 -> 27.2 mm, vias 8 -> 4
- net IFOUT3-: track 74.1 -> 1.89 mm, vias 4 -> 0
- net SCK: track 98.6 -> 27.1 mm, vias 5 -> 3
- net NSS3: track 73.4 -> 3.18 mm
- net IFOUT1+: track 69.5 -> 0.04 mm, vias 1 -> 0
- net IFOUT2+: track 67.8 -> 0.36 mm, vias 2 -> 0
- net +1V8: track 76.0 -> 8.56 mm, vias 2 -> 0
- net IFOUT1-: track 66.2 -> 0.04 mm, vias 1 -> 0
- net IFOUT2-: track 64.6 -> 0.36 mm, vias 2 -> 0
- net +5V: track 53.7 -> 0.00 mm, vias 2 -> 0
- net NSS4: track 52.5 -> 4.56 mm
- net NSS: track 45.9 -> 0.10 mm, vias 2 -> 0
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- removed copper zone on F.Cu, net +5V
- removed copper zone on F.Cu, net RF4O+
- removed copper zone on F.Cu, net RF4O-
- removed copper zone on F.Cu, net RFO1+
- removed copper zone on F.Cu, net RFO1-
- removed copper zone on F.Cu, net RFO2+
- removed copper zone on F.Cu, net RFO2-
- removed copper zone on F.Cu, net RFO3+
- removed copper zone on F.Cu, net RFO3-
- removed copper zone on F.Cu, net VPOS4R

Commit message: Silkscreen finishing
Silkscreen finishting
Parts:
- removed C17, C19: 1u, Capacitor_SMD:C_0603_1608Metric_Pad1.08x0.95mm_HandSolder
- removed C21, C24: 22u, Capacitor_SMD:C_0603_1608Metric_Pad1.08x0.95mm_HandSolder
- removed D4: ESD131-B1-W0201, Diode_SMD:Infineon_SG-WLL-2-3_0.58x0.28_P0.36mm
- removed D7: Green, LED_SMD:LED_0603_1608Metric_Pad1.05x0.95mm_HandSolder
- removed J2: Conn_01x04_Pin, Connector_PinHeader_2.54mm:PinHeader_1x04_P2.54mm_Vertical
- removed L2: 10n, Inductor_SMD:L_APV_ANR6020
- removed U3: USBLC6-2SC6, Package_TO_SOT_SMD:SOT-23-6_Handsoldering
- removed U6: HT7533-1, Package_TO_SOT_SMD:SOT-89-3_Handsoldering
- added C44: 10pF, Capacitor_SMD:C_0603_1608Metric_Pad1.08x0.95mm_HandSolder, F.Cu at (82.1, 129.5)
- added C45: 10 uF, Capacitor_SMD:C_0603_1608Metric_Pad1.08x0.95mm_HandSolder, F.Cu at (76.9, 115.6)
- added C46: 10uF, Capacitor_SMD:C_0603_1608Metric_Pad1.08x0.95mm_HandSolder, F.Cu at (79.5, 107.4)
- added C47: 4.7uF, Capacitor_SMD:C_0603_1608Metric_Pad1.08x0.95mm_HandSolder, F.Cu at (81.1, 107.3)
- added C48: 10uF, Capacitor_SMD:C_0603_1608Metric_Pad1.08x0.95mm_HandSolder, F.Cu at (76.8, 106.9)
- added C49: 0.01uF, Capacitor_SMD:C_0603_1608Metric_Pad1.08x0.95mm_HandSolder, F.Cu at (76.8, 105.0)
- added C50: 0.01uF, Capacitor_SMD:C_0603_1608Metric_Pad1.08x0.95mm_HandSolder, F.Cu at (76.8, 103.0)
- added C51: 10uF, Capacitor_SMD:C_0603_1608Metric_Pad1.08x0.95mm_HandSolder, F.Cu at (76.8, 101.3)
- added C52: 10 uF, Capacitor_SMD:C_0603_1608Metric_Pad1.08x0.95mm_HandSolder, F.Cu at (91.8, 111.0)
- added C53: 22uF, Capacitor_SMD:C_0603_1608Metric_Pad1.08x0.95mm_HandSolder, F.Cu at (93.2, 117.6)
- added C54: 4.7uF, Capacitor_SMD:C_0603_1608Metric_Pad1.08x0.95mm_HandSolder, F.Cu at (89.4, 105.7)
- added C55: 10uF, Capacitor_SMD:C_0603_1608Metric_Pad1.08x0.95mm_HandSolder, F.Cu at (88.2, 110.7)
- added C56: 1uF, Capacitor_SMD:C_0603_1608Metric_Pad1.08x0.95mm_HandSolder, F.Cu at (81.3, 86.5)
- added C59: pF, Capacitor_SMD:C_0603_1608Metric_Pad1.08x0.95mm_HandSolder, F.Cu at (83.0, 75.4)
- added C60: 10pF, Capacitor_SMD:C_0603_1608Metric_Pad1.08x0.95mm_HandSolder, F.Cu at (84.5, 75.4)
- added C61: 10pF, Capacitor_SMD:C_0603_1608Metric_Pad1.08x0.95mm_HandSolder, F.Cu at (86.1, 75.5)
- added C62: 10pF, Capacitor_SMD:C_0603_1608Metric_Pad1.08x0.95mm_HandSolder, F.Cu at (87.9, 75.5)
- added C63: 1uF, Capacitor_SMD:C_0603_1608Metric_Pad1.08x0.95mm_HandSolder, F.Cu at (71.6, 86.6)
- added C64: 1000pF, Capacitor_SMD:C_0603_1608Metric_Pad1.08x0.95mm_HandSolder, F.Cu at (64.6, 81.8)
- added C65: 0.01uF, Capacitor_SMD:C_0603_1608Metric_Pad1.08x0.95mm_HandSolder, F.Cu at (54.2, 80.4)
- added C66: 1uF, Capacitor_SMD:C_0603_1608Metric_Pad1.08x0.95mm_HandSolder, F.Cu at (56.3, 80.5)
- added C67: DNP, Capacitor_SMD:C_0603_1608Metric_Pad1.08x0.95mm_HandSolder, B.Cu at (71.5, 90.2)
- added C68: 0.018uF, Capacitor_SMD:C_0603_1608Metric_Pad1.08x0.95mm_HandSolder, B.Cu at (71.3, 97.0)
- added C69: 330pF, Capacitor_SMD:C_0603_1608Metric_Pad1.08x0.95mm_HandSolder, B.Cu at (78.0, 97.7)
- added C70: 220pF, Capacitor_SMD:C_0603_1608Metric_Pad1.08x0.95mm_HandSolder, B.Cu at (74.9, 97.0)
- added D1: Green, LED_SMD:LED_0603_1608Metric_Pad1.05x0.95mm_HandSolder, F.Cu at (73.0, 109.0)
- added FB1: FerriteBead, Inductor_SMD:L_0603_1608Metric_Pad1.05x0.95mm_HandSolder, F.Cu at (74.4, 103.9)
- added J1: Conn_01x04_Pin, Connector_PinHeader_2.54mm:PinHeader_1x04_P2.54mm_Vertical, F.Cu at (39.0, 65.8)
- added J13: Conn_Coaxial, Connector_Coaxial:SMA_Amphenol_132289_EdgeMount, F.Cu at (84.4, 42.2)
- added J14: Conn_01x05_Pin, Connector_PinHeader_2.54mm:PinHeader_1x05_P2.54mm_Vertical, F.Cu at (39.0, 77.8)
- added J16: Conn_Coaxial, Connector_Coaxial:SMA_Amphenol_132289_EdgeMount, F.Cu at (53.5, 42.5)
- added J17: Conn_Coaxial, Connector_Coaxial:SMA_Amphenol_132289_EdgeMount, F.Cu at (68.5, 42.4)
- added J5: Conn_01x05_Pin, Connector_PinHeader_2.54mm:PinHeader_1x05_P2.54mm_Vertical, F.Cu at (38.9, 61.1)
- added J6: RJ45_Shielded, Connector_RJ:RJ45_Amphenol_RJHSE5380, F.Cu at (40.0, 97.1)
- added J7: Barrel_Jack_Switch, Connector_BarrelJack:BarrelJack_Horizontal, F.Cu at (67.0, 131.4)
- added L7: 7.4nH, Inductor_SMD:L_0603_1608Metric_Pad1.05x0.95mm_HandSolder, F.Cu at (83.6, 77.0)
- added L8: 7.4nH, Inductor_SMD:L_0603_1608Metric_Pad1.05x0.95mm_HandSolder, F.Cu at (87.0, 77.0)
- added R18: 33.2k, Resistor_SMD:R_0603_1608Metric_Pad0.98x0.95mm_HandSolder, F.Cu at (88.6, 108.5)
- added R19: 0, Resistor_SMD:R_0603_1608Metric_Pad0.98x0.95mm_HandSolder, F.Cu at (85.2, 108.4)
- added R20: 0, Resistor_SMD:R_0603_1608Metric_Pad0.98x0.95mm_HandSolder, F.Cu at (87.1, 104.8)
- added R21: 0, Resistor_SMD:R_0603_1608Metric_Pad0.98x0.95mm_HandSolder, F.Cu at (85.2, 104.7)
- added R22: 0, Resistor_SMD:R_0603_1608Metric_Pad0.98x0.95mm_HandSolder, F.Cu at (76.9, 88.8)
- added R25: 51, Resistor_SMD:R_0603_1608Metric_Pad0.98x0.95mm_HandSolder, F.Cu at (63.9, 84.8)
- added R26: 100, Resistor_SMD:R_0603_1608Metric_Pad0.98x0.95mm_HandSolder, F.Cu at (61.9, 82.7)
- added R27: 0, Resistor_SMD:R_0603_1608Metric_Pad0.98x0.95mm_HandSolder, F.Cu at (59.3, 81.8)
- added R28: 0, Resistor_SMD:R_0603_1608Metric_Pad0.98x0.95mm_HandSolder, F.Cu at (54.2, 84.0)
- added R29: DNP, Resistor_SMD:R_0603_1608Metric_Pad0.98x0.95mm_HandSolder, F.Cu at (55.0, 88.0)
- added R3: 0, Resistor_SMD:R_0603_1608Metric_Pad0.98x0.95mm_HandSolder, F.Cu at (76.9, 108.4)
- added R30: 91, Resistor_SMD:R_0603_1608Metric_Pad0.98x0.95mm_HandSolder, B.Cu at (74.0, 89.2)
- added R31: 0, Resistor_SMD:R_0603_1608Metric_Pad0.98x0.95mm_HandSolder, B.Cu at (74.0, 92.7)
- added R32: 400, Resistor_SMD:R_0603_1608Metric_Pad0.98x0.95mm_HandSolder, B.Cu at (73.1, 95.3)
- added R33: 200, Resistor_SMD:R_0603_1608Metric_Pad0.98x0.95mm_HandSolder, B.Cu at (75.4, 98.6)
- added R34: 0, Resistor_SMD:R_0603_1608Metric_Pad0.98x0.95mm_HandSolder, F.Cu at (78.6, 115.5)
- added R4: 0, Resistor_SMD:R_0603_1608Metric_Pad0.98x0.95mm_HandSolder, F.Cu at (80.2, 104.9)
- added R5: 0, Resistor_SMD:R_0603_1608Metric_Pad0.98x0.95mm_HandSolder, F.Cu at (80.2, 103.0)
- added R6: 33.2k, Resistor_SMD:R_0603_1608Metric_Pad0.98x0.95mm_HandSolder, F.Cu at (82.7, 107.3)
- added R7: 470, Resistor_SMD:R_0603_1608Metric_Pad0.98x0.95mm_HandSolder, F.Cu at (71.1, 109.0)
- added R8: 0, Resistor_SMD:R_0603_1608Metric_Pad0.98x0.95mm_HandSolder, F.Cu at (89.6, 117.6)
- added TP1: TestPoint_Probe, TestPoint:TestPoint_Loop_D2.50mm_Drill1.0mm, F.Cu at (76.7, 111.2)
- added TP2: TestPoint_Probe, TestPoint:TestPoint_Loop_D2.50mm_Drill1.0mm, F.Cu at (85.2, 112.7)
- added U10: LT3045xDD, Package_DFN_QFN:DFN-10-1EP_3x3mm_P0.5mm_EP1.65x2.38mm, F.Cu at (89.9, 114.3)
- added U8: LT3045xDD, Package_DFN_QFN:DFN-10-1EP_3x3mm_P0.5mm_EP1.65x2.38mm, F.Cu at (80.5, 111.5)
- added Y2: ASE-xxxMHz, Oscillator:Oscillator_SMD_Abracon_ASE-4Pin_3.2x2.5mm, F.Cu at (57.8, 85.0)
- C1: value 10u -> 1uF
- C2: value 10u -> 0.01uF
- C29: moved to B.Cu
- J15: value RJ45 -> Conn_Coaxial; footprint Connector_RJ:RJ45_Amphenol_54602-x08_Horizontal -> Connector_Coaxial:SMA_Amphenol_132289_EdgeMount
- R17: value 1k -> 0
- SW1: value SW_Nidec_CAS-120A1 -> SW_SPDT; footprint Button_Switch_SMD:Nidec_Copal_CAS-120A -> Button_Switch_THT:SW_Slide_SPDT_Straight_CK_OS102011MS2Q
- moved R16 334.0 mm to (38.8, 129.2)
- moved SW1 332.4 mm to (56.0, 136.7), turned to 180 degrees
- moved R12 331.8 mm to (38.9, 112.1)
- moved U4 325.6 mm to (56.3, 112.2), turned to 90 degrees
- moved J8 323.5 mm to (39.0, 120.4), turned to -90 degrees
- moved U5 320.9 mm to (56.1, 126.5)
- moved R15 320.0 mm to (50.0, 112.2), turned to 90 degrees
- moved R10 319.6 mm to (47.1, 119.8)
- moved R11 319.4 mm to (47.1, 121.3)
- moved L3 318.7 mm to (59.2, 119.6), turned to -90 degrees
- moved D6 318.1 mm to (38.8, 127.1)
- moved D2 317.1 mm to (38.9, 114.1)
- moved C22 315.1 mm to (54.1, 122.8)
- moved R9 314.8 mm to (64.8, 109.9), turned to 180 degrees
- moved R13 313.5 mm to (66.5, 115.6), turned to -90 degrees
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Connections:
- C1 pad 1: VCC -> VCC_VCO
- C16 pad 1: /Power/V_PREfilt -> VSWITCH
- C2 pad 1: Net-(U9-REFP) -> GND
- C2 pad 2: unconnected-(C2-Pad2) -> REFN
- C3 pad 1: GND -> Net-(C3-Pad2)
- C3 pad 2: Net-(U9-REFN) -> REFN
- C4 pad 1: VCC -> VCC_LDO_3V
- J15 pad 1: IFOUT1+ -> Net-(J15-In)
- J15 pad 2: IFOUT1- -> GND
- J8 pad A6: /Power/usbc_d+ -> unconnected-(J8-D+-PadA6)
- J8 pad A7: /Power/usbc_d- -> unconnected-(J8-D--PadA7)
- J8 pad B6: /Power/usbc_d+ -> unconnected-(J8-D+-PadB6)
- J8 pad B7: /Power/usbc_d- -> unconnected-(J8-D--PadB7)
- R17 pad 2: GND -> VSWITCH
- SW1 pad 1: unconnected-(SW1-C-Pad1) -> +20V
- SW1 pad 2: /Power/V_PREfilt -> VSWITCH
- U1 pad 10: RFIN3+ -> GND
- U1 pad 11: RFIN3- -> GND
- U1 pad 15: RFIN4+ -> GND
- U1 pad 16: RFIN4- -> GND
- U1 pad 28: Net-(J14-Pin_2) -> unconnected-(U1-RXRST-Pad28)
- U1 pad 29: Net-(J14-Pin_3) -> unconnected-(U1-RXADV-Pad29)
- U1 pad 3: RFIN2- -> GND
- U1 pad 30: Net-(J14-Pin_4) -> unconnected-(U1-MRST-Pad30)
- U1 pad 31: Net-(J14-Pin_5) -> unconnected-(U1-MADV-Pad31)
- U1 pad 4: RFIN2+ -> GND
- U1 pad 46: RFIN1- -> GND
- U1 pad 47: RFIN1+ -> GND
- U4 pad 6: unconnected-(U4-Thermal_Pad-Pad6) -> GND
- U5 pad 2: /Power/V_PREfilt -> VSWITCH
- U5 pad 3: /Power/V_PREfilt -> VSWITCH
- U7 pad 10: MADV -> unconnected-(U7A-MADV-Pad10)
- U7 pad 11: MRST -> unconnected-(U7A-MRST-Pad11)
- U7 pad 8: TXADV -> unconnected-(U7A-TXADV-Pad8)
- U7 pad 9: TXRST -> unconnected-(U7A-TXRST-Pad9)
- U9 pad 14: VCC -> VCC_3V
- U9 pad 15: VCC -> VCC_3V
- U9 pad 16: VCC -> VCC_3V
- U9 pad 17: VCC -> VCC_3V
- U9 pad 21: VCC -> VCC_3V
- U9 pad 29: VCC -> VCC_3V
- U9 pad 30: VCC -> VCC_3V
- U9 pad 31: VCC -> VCC_3V
- U9 pad 32: VCC -> VCC_3V
- U9 pad 38: VCC -> VCC_LDO_3V
- U9 pad 39: VCC -> VCC_3V
- U9 pad 4: VCC -> VCC_3V
- U9 pad 41: Net-(J7-Pin_1) -> unconnected-(U9-MUXOUT-Pad41)
- U9 pad 43: Net-(U9-REFP) -> REFP
- U9 pad 44: Net-(U9-REFN) -> REFN
- U9 pad 45: VCC -> VCC_LDO_3V
- U9 pad 46: VCC -> VCC_LDO_3V
- U9 pad 47: VCC -> VCC_LDO_3V
- U9 pad 6: VCC -> Net-(U9-VCC_REG_OUT)
- U9 pad 7: VCC -> VCC_VCO
- U9 pad 8: +5V -> VCC_LDO
Routing:
- net GND: track 235.3 -> 501.8 mm, vias 620 -> 1085
- net VPOS4R: track 36.8 -> 261.4 mm, vias 0 -> 11
- net SCK: track 27.1 -> 209.1 mm, vias 3 -> 4
- net MOSI: track 27.2 -> 190.7 mm, vias 4 -> 7
- net +1V8: track 8.56 -> 150.8 mm, vias 0 -> 4
- net IFOUT3-: track 1.89 -> 143.2 mm, vias 0 -> 2
- net IFOUT3+: track 2.26 -> 143.2 mm, vias 0 -> 2
- net VCC_3V: track 0.00 -> 137.7 mm, vias 0 -> 9
- net MISO: track 31.7 -> 146.2 mm, vias 4 -> 5
- net IFOUT2+: track 0.36 -> 82.1 mm, vias 0 -> 3
- net IFOUT2-: track 0.36 -> 81.8 mm, vias 0 -> 3
- net IFOUT1-: track 0.04 -> 72.3 mm, vias 0 -> 3
- net IFOUT1+: track 0.04 -> 68.9 mm, vias 0 -> 3
- net NSS4: track 4.56 -> 72.2 mm
- net IFOUT4-: track 26.2 -> 90.3 mm, vias 0 -> 4
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- added copper zone on F.Cu, net +1V8
- added copper zone on F.Cu, net +20V
- added copper zone on F.Cu, net +3.3V
- added copper zone on F.Cu, net /Power/BST
- added copper zone on F.Cu, net /Power/SW
- added copper zone on F.Cu, net Net-(C53-Pad1)
- added copper zone on F.Cu, net Net-(D1-A)
- added copper zone on F.Cu, net Net-(R19-Pad2)
- added copper zone on F.Cu, net Net-(U10-EN/UV)
- added copper zone on F.Cu, net Net-(U10-OUT)
- added copper zone on F.Cu, net Net-(U10-SET)
- added copper zone on F.Cu, net Net-(U8-EN/UV)
- added copper zone on F.Cu, net VBUS
- added copper zone on F.Cu, net VCC_3V
- added copper zone on F.Cu, net VSWITCH
- added copper zone on In2.Cu, net VSWITCH
Other:
- board text added: "+1.8V"
- board text added: "+20V IN"
- board text added: "+3.3V"
- board text added: "20V"
- board text added: "62.5MHz-8GHz RFOUT+"
- board text added: "62.5MHz-8GHz RFOUT-"
- board text added: "8-16GHz RFOUT+"
- board text added: "8-16GHz RFOUT-"
- board text added: "Flatrim Dreshaj Justin Adrowski Durotimi Johnson EE418 Phased Array FMCW Radar 26-32GHz"
- board text added: "GND"
- board text added: "NSS SCK MISO MOSI"
- board text added: "NSS3 NSS4"
- board text added: "RFOUT -+"
- board text added: "RFOUT1 +-"
- board text added: "RFOUT2 +-"
- board text added: "RFOUT3 -+"
- board text added: "RFOUT4 -+"
- board text added: "VBUS"
- board text added: "VBUS 5V"
- board text added: "VCO TUNE"
- board text removed: "RF 4 -+"
- board text removed: "RF1 +-"
- board text removed: "RF2 +-"
- board text removed: "RF3 -+"
- board text removed: "RFIN4 -+"

Commit message: final changes to RF board
final changes to RF board + grbs
Parts:
- moved J7 0.40 mm to (67.0, 131.0)
- moved J3 0.28 mm to (79.6, 135.2)
Routing:
- net GND: vias 1085 -> 1542
Other:
- board text added: "RFIN1 +-"
- board text added: "RFIN4 -+"
- board text removed: "RFIN4 +-"
- board text removed: "RFOUT -+"
