File: fmcw_radar_sch/Up_Down_Converter/biasing.kicad_sch (KiCad schematic)
At the start: 18 parts, among them J13 Conn_Coaxial, J15 Conn_Coaxial, J16 Conn_Coaxial, J17 Conn_Coaxial

Commit message: Silkscreen finishing
Silkscreen finishting
Parts:
- removed C42, C43, C58: 10pF, symbol Device:C
- removed C57: pF, symbol Device:C
- removed L5, L6: 7.4nH, symbol Device:L
- removed R23, R24: 50, symbol Device:R
- C59, C60, C61, C62: footprint (none) -> Capacitor_SMD:C_0603_1608Metric_Pad1.08x0.95mm_HandSolder
- J13, J15, J16, J17: footprint (none) -> Connector_Coaxial:SMA_Amphenol_132289_EdgeMount
- L7, L8: footprint (none) -> Inductor_SMD:L_0603_1608Metric_Pad1.05x0.95mm_HandSolder

Commit message: changes from yesterday
changes from yesterday
Parts:
- C59: value pF -> 10 pF; footprint Capacitor_SMD:C_0603_1608Metric_Pad1.08x0.95mm_HandSolder -> Capacitor_SMD:C_0402_1005Metric_Pad0.74x0.62mm_HandSolder
- C60, C61, C62: footprint Capacitor_SMD:C_0603_1608Metric_Pad1.08x0.95mm_HandSolder -> Capacitor_SMD:C_0402_1005Metric_Pad0.74x0.62mm_HandSolder
- J13, J15, J16, J17: footprint Connector_Coaxial:SMA_Amphenol_132289_EdgeMount -> RF_extra:BEL_142-1701-831
- L7, L8: footprint Inductor_SMD:L_0603_1608Metric_Pad1.05x0.95mm_HandSolder -> Capacitor_SMD:C_0402_1005Metric_Pad0.74x0.62mm_HandSolder
Other:
- moved on the sheet: C62, J13
Changed lines of the file:
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@@
 	)
 	(junction
-		(at 185.42 52.07)
+		(at 187.96 52.07)
 		(diameter 0)
 		(color 0 0 0 0)
@@
 	(wire
 		(pts
-			(xy 153.67 76.2) (xy 148.59 76.2)
+			(xy 158.75 74.93) (xy 158.75 71.12)
+		)
+		(stroke
+			(width 0)
+			(type default)
+		)
+	)
+	(wire
+		(pts
+			(xy 153.67 80.01) (xy 151.13 80.01)
 		)
 		(stroke
@@
 	(wire
 		(pts
-			(xy 185.42 60.96) (xy 185.42 63.5)
+			(xy 187.96 60.96) (xy 187.96 63.5)
 		)
 		(stroke
@@
 	(wire
 		(pts
-			(xy 185.42 52.07) (xy 185.42 39.37)
+			(xy 187.96 52.07) (xy 187.96 39.37)
 		)
 		(stroke
@@
 	(wire
 		(pts
+			(xy 181.61 52.07) (xy 187.96 52.07)
+		)
+		(stroke
+			(width 0)
+			(type default)
+		)
+	)
+	(wire
+		(pts
 			(xy 170.18 30.48) (xy 170.18 52.07)
 		)
@@
 	(wire
 		(pts
-			(xy 148.59 76.2) (xy 148.59 77.47)
-		)
-		(stroke
-			(width 0)
-			(type default)
-		)
-	)
-	(wire
-		(pts
-			(xy 185.42 53.34) (xy 185.42 52.07)
+			(xy 151.13 80.01) (xy 151.13 81.28)
+		)
+		(stroke
+			(width 0)
+			(type default)
+		)
+	)
+	(wire
+		(pts
+			(xy 187.96 53.34) (xy 187.96 52.07)
 		)
 		(stroke
@@
 		(pts
 			(xy 203.2 46.99) (xy 203.2 48.26)
-		)
-		(stroke
-			(width 0)
-			(type default)
-		)
-	)
-	(wire
-		(pts
-			(xy 181.61 52.07) (xy 185.42 52.07)
 		)
 		(stroke
@@
 	(symbol
 		(lib_id "power:GND")
-		(at 185.42 63.5 0)
+		(at 187.96 63.5 0)
 		(unit 1)
 		(exclude_from_sim no)
@@
 		(fields_autoplaced yes)
 		(property "Reference" "#PWR0165"
-			(at 185.42 69.85 0)
+			(at 187.96 69.85 0)
 			(effects
 				(font
@@
 		)
 		(property "Value" "GND"
-			(at 185.42 68.58 0)
+			(at 187.96 68.58 0)
 			(effects
 				(font
@@
 		)
 		(property "Footprint" ""
-			(at 185.42 63.5 0)
+			(at 187.96 63.5 0)
 			(effects
 				(font
@@
 		)
 		(property "Datasheet" ""
-			(at 185.42 63.5 0)
+			(at 187.96 63.5 0)
 			(effects
 				(font
@@
 		)
 		(property "Description" "Power symbol creates a global label with name \"GND\" , ground"
-			(at 185.42 63.5 0)
+			(at 187.96 63.5 0)
 			(effects
 				(font
@@
 	(symbol
 		(lib_id "power:GND")
-		(at 148.59 77.47 0)
+		(at 151.13 81.28 0)
 		(unit 1)
 		(exclude_from_sim no)
@@
 		(fields_autoplaced yes)
 		(property "Reference" "#PWR0163"
-			(at 148.59 83.82 0)
+			(at 151.13 87.63 0)
 			(effects
 				(font
@@
 		)
 		(property "Value" "GND"
-			(at 148.59 82.55 0)
+			(at 151.13 86.36 0)
 			(effects
 				(font
@@
 		)
 		(property "Footprint" ""
-			(at 148.59 77.47 0)
+			(at 151.13 81.28 0)
 			(effects
 				(font
@@
 		)
 		(property "Datasheet" ""
-			(at 148.59 77.47 0)
+			(at 151.13 81.28 0)
 			(effects
 				(font
@@
 		)
 		(property "Description" "Power symbol creates a global label with name \"GND\" , ground"
-			(at 148.59 77.47 0)
+			(at 151.13 81.28 0)
 			(effects
 				(font
@@
 			)
 		)
-		(property "Footprint" "Capacitor_SMD:C_0603_1608Metric_Pad1.08x0.95mm_HandSolder"
+		(property "Footprint" "Capacitor_SMD:C_0402_1005Metric_Pad0.74x0.62mm_HandSolder"
 			(at 171.1452 71.12 0)
 			(effects
@@
 			)
 		)
-		(property "Footprint" "Connector_Coaxial:SMA_Amphenol_132289_EdgeMount"
+		(property "Footprint" "RF_extra:BEL_142-1701-831"
 			(at 231.14 49.53 0)
 			(effects
@@
 			)
 		)
-		(property "Value" "pF"
+		(property "Value" "10 pF"
 			(at 135.89 60.9599 0)
 			(effects
@@
 			)
 		)
-		(property "Footprint" "Capacitor_SMD:C_0603_1608Metric_Pad1.08x0.95mm_HandSolder"
+		(property "Footprint" "Capacitor_SMD:C_0402_1005Metric_Pad0.74x0.62mm_HandSolder"
 			(at 133.0452 63.5 0)
 			(effects
@@
 	(symbol
 		(lib_id "Device:C")
-		(at 185.42 57.15 0)
+		(at 187.96 57.15 0)
 		(unit 1)
 		(exclude_from_sim no)
@@
 		(fields_autoplaced yes)
 		(property "Reference" "C62"
-			(at 189.23 55.8799 0)
+			(at 191.77 55.8799 0)
 			(effects
 				(font
@@
 		)
 		(property "Value" "10pF"
-			(at 189.23 58.4199 0)
-			(effects
-				(font
-					(size 1.27 1.27)
-				)
-				(justify left)
-			)
-		)
-		(property "Footprint" "Capacitor_SMD:C_0603_1608Metric_Pad1.08x0.95mm_HandSolder"
-			(at 186.3852 60.96 0)
+			(at 191.77 58.4199 0)
+			(effects
+				(font
+					(size 1.27 1.27)
+				)
+				(justify left)
+			)
+		)
+		(property "Footprint" "Capacitor_SMD:C_0402_1005Metric_Pad0.74x0.62mm_HandSolder"
+			(at 188.9252 60.96 0)
 			(effects
 				(font
@@
 		)
 		(property "Datasheet" "~"
-			(at 185.42 57.15 0)
+			(at 187.96 57.15 0)
 			(effects
 				(font
@@
 		)
 		(property "Description" "Unpolarized capacitor"
-			(at 185.42 57.15 0)
+			(at 187.96 57.15 0)
 			(effects
 				(font
@@
 			)
 		)
-		(property "Footprint" "Capacitor_SMD:C_0603_1608Metric_Pad1.08x0.95mm_HandSolder"
+		(property "Footprint" "Capacitor_SMD:C_0402_1005Metric_Pad0.74x0.62mm_HandSolder"
 			(at 159.7152 71.12 0)
 			(effects
@@
 			)
 		)
-		(property "Footprint" "Connector_Coaxial:SMA_Amphenol_132289_EdgeMount"
+		(property "Footprint" "RF_extra:BEL_142-1701-831"
 			(at 170.18 83.82 0)
 			(effects
@@
 			)
 		)
-		(property "Footprint" "Inductor_SMD:L_0603_1608Metric_Pad1.05x0.95mm_HandSolder"
+		(property "Footprint" "Capacitor_SMD:C_0402_1005Metric_Pad0.74x0.62mm_HandSolder"
 			(at 177.8 52.07 0)
 			(effects
@@
 			)
 		)
-		(property "Footprint" "Inductor_SMD:L_0603_1608Metric_Pad1.05x0.95mm_HandSolder"
+		(property "Footprint" "Capacitor_SMD:C_0402_1005Metric_Pad0.74x0.62mm_HandSolder"
 			(at 142.24 52.07 0)
 			(effects
@@
 	(symbol
 		(lib_id "power:VDD")
-		(at 185.42 39.37 0)
+		(at 187.96 39.37 0)
 		(unit 1)
 		(exclude_from_sim no)
@@
 		(fields_autoplaced yes)
 		(property "Reference" "#PWR0164"
-			(at 185.42 43.18 0)
+			(at 187.96 43.18 0)
 			(effects
 				(font
@@
 		)
 		(property "Value" "VDD_X1"
-			(at 185.42 34.29 0)
+			(at 187.96 34.29 0)
 			(effects
 				(font
@@
 		)
 		(property "Footprint" ""
-			(at 185.42 39.37 0)
+			(at 187.96 39.37 0)
 			(effects
 				(font
@@
 		)
 		(property "Datasheet" ""
-			(at 185.42 39.37 0)
+			(at 187.96 39.37 0)
 			(effects
 				(font
@@
 		)
 		(property "Description" "Power symbol creates a global label with name \"VDD\""
-			(at 185.42 39.37 0)
+			(at 187.96 39.37 0)
 			(effects
 				(font
@@
 			)
 		)
-		(property "Footprint" "Connector_Coaxial:SMA_Amphenol_132289_EdgeMount"
+		(property "Footprint" "RF_extra:BEL_142-1701-831"
 			(at 213.36 46.99 0)
 			(effects
@@
 	(symbol
 		(lib_id "Connector:Conn_Coaxial")
-		(at 158.75 76.2 270)
+		(at 158.75 80.01 270)
 		(unit 1)
 		(exclude_from_sim no)
@@
 		(fields_autoplaced yes)
 		(property "Reference" "J13"
-			(at 162.56 74.6124 90)
+			(at 162.56 78.4224 90)
 			(effects
 				(font
@@
 		)
 		(property "Value" "Conn_Coaxial"
-			(at 162.56 77.1524 90)
-			(effects
-				(font
-					(size 1.27 1.27)
-				)
-				(justify left)
-				(hide yes)
-			)
-		)
-		(property "Footprint" "Connector_Coaxial:SMA_Amphenol_132289_EdgeMount"
-			(at 158.75 76.2 0)
+			(at 162.56 80.9624 90)
+			(effects
+				(font
+					(size 1.27 1.27)
+				)
+				(justify left)
+				(hide yes)
+			)
+		)
+		(property "Footprint" "RF_extra:BEL_142-1701-831"
+			(at 158.75 80.01 0)
 			(effects
 				(font
@@
 		)
 		(property "Datasheet" "~"
-			(at 158.75 76.2 0)
+			(at 158.75 80.01 0)
 			(effects
 				(font
@@
 		)
 		(property "Description" "coaxial connector (BNC, SMA, SMB, SMC, Cinch/RCA, LEMO, ...)"
-			(at 158.75 76.2 0)
-			(effects
-				(font
+			(at 158.75 80.01 0)
+			(effects
+				(font
