File: fmcw_radar_sch/Up_Down_Converter/power_up_down.kicad_sch (KiCad schematic)
At the start: 38 parts, among them J8 USB_C_Receptacle_USB2.0_16P, J9 Screw_Terminal_01x02, SW1 SW_Nidec_CAS-120A1, U2 LP3875EMP-2.5/NOPB, U3 USBLC6-2SC6, U4 TLV75718PDYDR, U5 AP63203WU, U6 HT7533-1

Commit message: layout
Parts:
- C12, C14, C15, C16, C18, C20, C22, C23: footprint Capacitor_SMD:C_1206_3216Metric_Pad1.33x1.80mm_HandSolder -> Capacitor_SMD:C_0603_1608Metric_Pad1.08x0.95mm_HandSolder
- C13: footprint Capacitor_SMD:C_0603_1608Metric -> Capacitor_SMD:C_0603_1608Metric_Pad1.08x0.95mm_HandSolder
- C17, C19, C21, C24: footprint Capacitor_SMD:C_0805_2012Metric -> Capacitor_SMD:C_0603_1608Metric_Pad1.08x0.95mm_HandSolder
Changed lines of the file:
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@@
 			)
 		)
-		(property "Footprint" "Capacitor_SMD:C_0805_2012Metric"
+		(property "Footprint" "Capacitor_SMD:C_0603_1608Metric_Pad1.08x0.95mm_HandSolder"
 			(at 251.1552 87.63 0)
 			(effects
@@
 			)
 		)
-		(property "Footprint" "Capacitor_SMD:C_0805_2012Metric"
+		(property "Footprint" "Capacitor_SMD:C_0603_1608Metric_Pad1.08x0.95mm_HandSolder"
 			(at 284.1752 88.9 0)
 			(effects
@@
 			)
 		)
-		(property "Footprint" "Capacitor_SMD:C_0805_2012Metric"
+		(property "Footprint" "Capacitor_SMD:C_0603_1608Metric_Pad1.08x0.95mm_HandSolder"
 			(at 203.5048 92.71 0)
 			(effects
@@
 			)
 		)
-		(property "Footprint" "Capacitor_SMD:C_0805_2012Metric"
+		(property "Footprint" "Capacitor_SMD:C_0603_1608Metric_Pad1.08x0.95mm_HandSolder"
 			(at 236.5248 87.63 0)
 			(effects
@@
 			)
 		)
-		(property "Footprint" "Capacitor_SMD:C_1206_3216Metric_Pad1.33x1.80mm_HandSolder"
+		(property "Footprint" "Capacitor_SMD:C_0603_1608Metric_Pad1.08x0.95mm_HandSolder"
 			(at 200.66 36.83 0)
 			(effects
@@
 			)
 		)
-		(property "Footprint" "Capacitor_SMD:C_1206_3216Metric_Pad1.33x1.80mm_HandSolder"
+		(property "Footprint" "Capacitor_SMD:C_0603_1608Metric_Pad1.08x0.95mm_HandSolder"
 			(at 44.45 137.16 0)
 			(effects
@@
 			)
 		)
-		(property "Footprint" "Capacitor_SMD:C_1206_3216Metric_Pad1.33x1.80mm_HandSolder"
+		(property "Footprint" "Capacitor_SMD:C_0603_1608Metric_Pad1.08x0.95mm_HandSolder"
 			(at 121.92 134.62 0)
 			(effects
@@
 			)
 		)
-		(property "Footprint" "Capacitor_SMD:C_1206_3216Metric_Pad1.33x1.80mm_HandSolder"
+		(property "Footprint" "Capacitor_SMD:C_0603_1608Metric_Pad1.08x0.95mm_HandSolder"
 			(at 261.62 36.83 0)
 			(effects
@@
 			)
 		)
-		(property "Footprint" "Capacitor_SMD:C_0603_1608Metric"
+		(property "Footprint" "Capacitor_SMD:C_0603_1608Metric_Pad1.08x0.95mm_HandSolder"
 			(at 85.09 43.4848 0)
 			(effects
@@
 			)
 		)
-		(property "Footprint" "Capacitor_SMD:C_1206_3216Metric_Pad1.33x1.80mm_HandSolder"
+		(property "Footprint" "Capacitor_SMD:C_0603_1608Metric_Pad1.08x0.95mm_HandSolder"
 			(at 215.5952 133.35 0)
 			(effects
@@
 			)
 		)
-		(property "Footprint" "Capacitor_SMD:C_1206_3216Metric_Pad1.33x1.80mm_HandSolder"
+		(property "Footprint" "Capacitor_SMD:C_0603_1608Metric_Pad1.08x0.95mm_HandSolder"
 			(at 163.5252 132.08 0)
 			(effects
@@
 			)
 		)
-		(property "Footprint" "Capacitor_SMD:C_1206_3216Metric_Pad1.33x1.80mm_HandSolder"
+		(property "Footprint" "Capacitor_SMD:C_0603_1608Metric_Pad1.08x0.95mm_HandSolder"
 			(at 270.51 36.83 0)
 			(effects
@@
 			)
 		)
-		(property "Footprint" "Capacitor_SMD:C_1206_3216Metric_Pad1.33x1.80mm_HandSolder"
+		(property "Footprint" "Capacitor_SMD:C_0603_1608Metric_Pad1.08x0.95mm_HandSolder"
 			(at 245.11 31.75 0)
 			(effects

Commit message: changes
changes
Parts:
- U2: footprint nonkicad:MP05A -> RF_extra:DNT12_TEX
- U4: footprint nonkicad:DYD0005A-MFG -> RF_extra:DYD0005A-MFG
Changed lines of the file:
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@@
 			)
 		)
-		(property "Footprint" "nonkicad:DYD0005A-MFG"
+		(property "Footprint" "RF_extra:DYD0005A-MFG"
 			(at 170.18 123.19 0)
 			(effects
@@
 			)
 		)
-		(property "Footprint" "nonkicad:MP05A"
+		(property "Footprint" "RF_extra:DNT12_TEX"
 			(at 49.53 123.19 0)
 			(effects

Commit message: a lot of updates
usb power delivery + finishing touches
Parts:
- removed C17, C19: 1u, Capacitor_SMD:C_0603_1608Metric_Pad1.08x0.95mm_HandSolder, symbol Device:C
- removed C21, C24: 22u, Capacitor_SMD:C_0603_1608Metric_Pad1.08x0.95mm_HandSolder, symbol Device:C
- removed D4: ESD131-B1-W0201, Diode_SMD:Infineon_SG-WLL-2-3_0.58x0.28_P0.36mm, symbol Diode:ESD131-B1-W0201
- removed D7: Green, LED_SMD:LED_0603_1608Metric_Pad1.05x0.95mm_HandSolder, symbol Device:LED
- removed J9: Screw_Terminal_01x02, TerminalBlock:TerminalBlock_MaiXu_MX126-5.0-02P_1x02_P5.00mm, symbol Connector:Screw_Terminal_01x02
- removed L2: 10n, Inductor_SMD:L_APV_ANR6020, symbol Device:L
- removed R17: 1k, Resistor_SMD:R_0603_1608Metric_Pad0.98x0.95mm_HandSolder, symbol Device:R
- removed SW1: SW_Nidec_CAS-120A1, Button_Switch_SMD:Nidec_Copal_CAS-120A, symbol Switch:SW_Nidec_CAS-120A1
- removed U6: HT7533-1, Package_TO_SOT_SMD:SOT-89-3_Handsoldering, symbol Regulator_Linear:HT75xx-1-SOT89
- added SW2: SW_DP3T, symbol Switch:SW_DP3T
Connections:
- net GND: now also U4.6 (Thermal_Pad)
- net VBUS: now also SW2.4
- net V_PREfilt renamed VSWITCH
- net VSWITCH: now also SW2.3
- new net +10V: SW2.2
- new net +20V: SW2.1
- no-connect marks 7 -> 6
Other:
- note removed: "+BATT from screw Connector(nom. +9V)"
- note removed: "3.3VA"
- note removed: "DCR=0R15"
- note removed: "VBUS from USB Connector(nom. +5V) Min. 22uF inp./outp. caps"
- moved on the sheet: C12, C14, C15, C18, D3, D5, R13, R14, R15, R9, U2, U4

Commit message: Silkscreen finishing
Silkscreen finishting
Parts:
- removed SW2: SW_DP3T, symbol Switch:SW_DP3T
- removed U3: USBLC6-2SC6, Package_TO_SOT_SMD:SOT-23-6_Handsoldering, symbol Power_Protection:USBLC6-2SC6
- added SW1: SW_SPDT, Button_Switch_THT:SW_Slide_SPDT_Straight_CK_OS102011MS2Q, symbol Switch:SW_SPDT
Connections:
- net +20V: now also SW1.1 (A)
- net VBUS: now also SW1.3 (C)
- net VSWITCH: now also SW1.2 (B)
- net usbc_d+: no longer names the net of J8.A6 (D+)
- net usbc_d+: no longer J8.B6 (D+)
- net usbc_d-: no longer names the net of J8.A7 (D-)
- net usbc_d-: no longer J8.B7 (D-)
- no-connect marks 6 -> 8

Commit message: changes from yesterday
changes from yesterday
Parts:
- C22, C23: footprint Capacitor_SMD:C_0603_1608Metric_Pad1.08x0.95mm_HandSolder -> Capacitor_SMD:C_1206_3216Metric_Pad1.33x1.80mm_HandSolder
- U2: footprint RF_extra:DNT12_TEX -> RF_extra:MP05A
Changed lines of the file:
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@@
 			)
 		)
-		(property "Footprint" "Capacitor_SMD:C_0603_1608Metric_Pad1.08x0.95mm_HandSolder"
+		(property "Footprint" "Capacitor_SMD:C_1206_3216Metric_Pad1.33x1.80mm_HandSolder"
 			(at 261.62 36.83 0)
 			(effects
@@
 			)
 		)
-		(property "Footprint" "RF_extra:DNT12_TEX"
+		(property "Footprint" "RF_extra:MP05A"
 			(at 58.42 121.92 0)
 			(effects
@@
 			)
 		)
-		(property "Footprint" "Capacitor_SMD:C_0603_1608Metric_Pad1.08x0.95mm_HandSolder"
+		(property "Footprint" "Capacitor_SMD:C_1206_3216Metric_Pad1.33x1.80mm_HandSolder"
 			(at 270.51 36.83 0)
 			(effects
