File: fmcw_radar_sch/Power_Delivery/Power_Delivery.kicad_pcb (KiCad board)
At the start: 2 copper layers, 100 x 100 mm, 52 parts, among them J1 USB_C_Receptacle_USB2.0_16P, J2 Screw_Terminal_01x03, J3 Conn_01x05_Pin, J4 Barrel_Jack_Switch, Q1 DMP3099L, Q2 DMP3099L, Q3 DMP3099L, Q4 DMP3099L, Q5 2N7002, U1 CYPD3177-24LQ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

Commit message: Silkscreen finishing
Silkscreen finishting
Routing:
- net GND: vias 251 -> 223
Other:
- board text added: "+20V 3A OUT +20V 5A OUT"
- board text added: "+3.3V"
- board text added: "Flatrim Dreshaj USBC Power Delivery 60 - 100W EE418 Phased Array FMCW Radar 26-32GHz"
- board text added: "GND +3.3V +5V SAFE"
- board text added: "SDA SCL INT GPIO1 +3.3V"
- board text added: "USBC-PD"

Commit message: final changes to RF board
final changes to RF board + grbs
Routing:
- net GND: vias 223 -> 231
Changed lines of the file:
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@@
 			(outputformat 1)
 			(mirror no)
-			(drillshape 1)
+			(drillshape 0)
 			(scaleselection 1)
-			(outputdirectory "")
+			(outputdirectory "pow_del_grbs/")
 		)
 	)
@@
 	)
 	(via
+		(at 150 95)
+		(size 0.6)
+		(drill 0.3)
+		(layers "F.Cu" "B.Cu")
+		(net 1)
+	)
+	(via
 		(at 109.22 88.9)
 		(size 0.6)
@@
 	)
 	(via
+		(at 148.2 94.075)
+		(size 0.6)
+		(drill 0.3)
+		(layers "F.Cu" "B.Cu")
+		(net 1)
+	)
+	(via
 		(at 157.48 81.28)
 		(size 0.6)
@@
 	)
 	(via
+		(at 149.08 94.86)
+		(size 0.6)
+		(drill 0.3)
+		(layers "F.Cu" "B.Cu")
+		(net 1)
+	)
+	(via
 		(at 187.96 55.88)
 		(size 0.6)
@@
 	)
 	(via
+		(at 148.175 95.675)
+		(size 0.6)
+		(drill 0.3)
+		(layers "F.Cu" "B.Cu")
+		(net 1)
+	)
+	(via
 		(at 182.88 60.96)
 		(size 0.6)
@@
 	)
 	(via
+		(at 149.975 95.7)
+		(size 0.6)
+		(drill 0.3)
+		(layers "F.Cu" "B.Cu")
+		(net 1)
+	)
+	(via
 		(at 101.6 111.76)
 		(size 0.6)
@@
 	)
 	(via
-		(at 149.08 94.86)
-		(size 0.6)
-		(drill 0.3)
-		(layers "F.Cu" "B.Cu")
-		(net 1)
-	)
-	(via
 		(at 137.16 127)
 		(size 0.6)
@@
 	)
 	(via
+		(at 149 94)
+		(size 0.6)
+		(drill 0.3)
+		(layers "F.Cu" "B.Cu")
+		(net 1)
+	)
+	(via
+		(at 150 94)
+		(size 0.6)
+		(drill 0.3)
+		(layers "F.Cu" "B.Cu")
+		(net 1)
+	)
+	(via
 		(at 110.49 87.63)
 		(size 0.6)
@@
 	)
 	(via
+		(at 149.05 95.675)
+		(size 0.6)
+		(drill 0.3)
+		(layers "F.Cu" "B.Cu")
+		(net 1)
+	)
+	(via
 		(at 172.72 96.52)
 		(size 0.6)
@@
 	)
 	(via
+		(at 148.2 94.925)
+		(size 0.6)
+		(drill 0.3)
+		(layers "F.Cu" "B.Cu")
+		(net 1)
+	)
+	(via
 		(at 167.64 127)
 		(size 0.6)
@@
 	)
 	(segment
-		(start 141.815 96.89)
-		(end 143.17 96.89)
+		(start 143.17 96.89)
+		(end 141.815 96.89)
 		(width 0.5)
 		(layer "F.Cu")
@@
 		(net 31)
 	)
-	(segment
-		(start 143.17 96.89)
-		(end 144.38 95.68)
-		(width 0.5)
-		(layer "F.Cu")
-		(net 31)
-	)
 	(via
 		(at 152.66 95.68462)
@@
 	)
 	(via
-		(at 144.38 95.68)
+		(at 143.17 96.89)
 		(size 0.6)
 		(drill 0.3)
@@
 	(segment
 		(start 151.93462 95.68462)
-		(end 151.93 95.68)
+		(end 152.66 95.68462)
 		(width 0.3)
 		(layer "B.Cu")
@@
 	)
 	(segment
-		(start 151.93 95.68)
-		(end 144.38 95.68)
+		(start 145.7 97)
+		(end 150.61924 97)
 		(width 0.3)
 		(layer "B.Cu")
@@
 	)
 	(segment
-		(start 152.66 95.68462)
+		(start 145.59 96.89)
+		(end 145.7 97)
+		(width 0.3)
+		(layer "B.Cu")
+		(net 31)
+	)
+	(segment
+		(start 150.61924 97)
 		(end 151.93462 95.68462)
 		(width 0.3)
 		(layer "B.Cu")
+		(net 31)
+	)
+	(segment
+		(start 143.17 96.89)
+		(end 145.59 96.89)
+		(width 0.3)
+		(layer "B.Cu")

Commit message: changes from yesterday
changes from yesterday
Parts:
- C11, C12: footprint Capacitor_SMD:C_0603_1608Metric -> Capacitor_SMD:C_1206_3216Metric
- moved C12 1.75 mm to (122.1, 64.0)
- moved C11 0.75 mm to (122.1, 66.9)
Routing:
- net GND: track 29.3 -> 30.9 mm
Changed lines of the file:
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@@
 		)
 	)
-	(footprint "Capacitor_SMD:C_0603_1608Metric"
+	(footprint "Capacitor_SMD:C_1206_3216Metric"
 		(layer "F.Cu")
-		(at 122.09 67.64 180)
-		(descr "Capacitor SMD 0603 (1608 Metric), square (rectangular) end terminal, IPC-7351 nominal, (Body size source: IPC-SM-782 page 76, https://www.pcb-3d.com/wordpress/wp-content/uploads/ipc-sm-782a_amendment_1_and_2.pdf), generated with kicad-footprint-generator")
+		(at 122.09 66.89 180)
+		(descr "Capacitor SMD 1206 (3216 Metric), square (rectangular) end terminal, IPC-7351 nominal, (Body size source: IPC-SM-782 page 76, https://www.pcb-3d.com/wordpress/wp-content/uploads/ipc-sm-782a_amendment_1_and_2.pdf), generated with kicad-footprint-generator")
 		(tags "capacitor")
 		(property "Reference" "C11"
-			(at 2.97 0 0)
+			(at 0 -1.85 180)
 			(layer "F.SilkS")
+			(hide yes)
 			(effects
 				(font
@@
 		)
 		(property "Value" "22uF"
-			(at 0 1.43 0)
+			(at 0 1.85 180)
 			(layer "F.Fab")
 			(effects
@@
 		)
 		(property "Datasheet" ""
-			(at 0 0 0)
+			(at 0 0 180)
 			(layer "F.Fab")
 			(hide yes)
@@
 		)
 		(property "Description" "Unpolarized capacitor, small symbol"
-			(at 0 0 0)
+			(at 0 0 180)
 			(layer "F.Fab")
 			(hide yes)
@@
 		(attr smd)
 		(fp_line
-			(start -0.14058 0.51)
-			(end 0.14058 0.51)
+			(start -0.711252 0.91)
+			(end 0.711252 0.91)
 			(stroke
 				(width 0.12)
@@
 		)
 		(fp_line
-			(start -0.14058 -0.51)
-			(end 0.14058 -0.51)
+			(start -0.711252 -0.91)
+			(end 0.711252 -0.91)
 			(stroke
 				(width 0.12)
@@
 		)
 		(fp_line
-			(start 1.48 0.73)
-			(end -1.48 0.73)
+			(start 2.3 1.15)
+			(end -2.3 1.15)
 			(stroke
 				(width 0.05)
@@
 		)
 		(fp_line
-			(start 1.48 -0.73)
-			(end 1.48 0.73)
+			(start 2.3 -1.15)
+			(end 2.3 1.15)
 			(stroke
 				(width 0.05)
@@
 		)
 		(fp_line
-			(start -1.48 0.73)
-			(end -1.48 -0.73)
+			(start -2.3 1.15)
+			(end -2.3 -1.15)
 			(stroke
 				(width 0.05)
@@
 		)
 		(fp_line
-			(start -1.48 -0.73)
-			(end 1.48 -0.73)
+			(start -2.3 -1.15)
+			(end 2.3 -1.15)
 			(stroke
 				(width 0.05)
@@
 		)
 		(fp_line
-			(start 0.8 0.4)
-			(end -0.8 0.4)
+			(start 1.6 0.8)
+			(end -1.6 0.8)
 			(stroke
 				(width 0.1)
@@
 		)
 		(fp_line
-			(start 0.8 -0.4)
-			(end 0.8 0.4)
+			(start 1.6 -0.8)
+			(end 1.6 0.8)
 			(stroke
 				(width 0.1)
@@
 		)
 		(fp_line
-			(start -0.8 0.4)
-			(end -0.8 -0.4)
+			(start -1.6 0.8)
+			(end -1.6 -0.8)
 			(stroke
 				(width 0.1)
@@
 		)
 		(fp_line
-			(start -0.8 -0.4)
-			(end 0.8 -0.4)
+			(start -1.6 -0.8)
+			(end 1.6 -0.8)
 			(stroke
 				(width 0.1)
@@
 		)
 		(fp_text user "${REFERENCE}"
-			(at 0 0 0)
+			(at 0 0 180)
 			(layer "F.Fab")
 			(effects
 				(font
-					(size 0.4 0.4)
-					(thickness 0.06)
+					(size 0.8 0.8)
+					(thickness 0.12)
 				)
 			)
 		)
 		(pad "1" smd roundrect
-			(at -0.775 0 180)
-			(size 0.9 0.95)
+			(at -1.475 0 180)
+			(size 1.15 1.8)
 			(layers "F.Cu" "F.Mask" "F.Paste")
-			(roundrect_rratio 0.25)
+			(roundrect_rratio 0.217391)
 			(net 1 "GND")
 			(pintype "passive")
 		)
 		(pad "2" smd roundrect
-			(at 0.775 0 180)
-			(size 0.9 0.95)
+			(at 1.475 0 180)
+			(size 1.15 1.8)
 			(layers "F.Cu" "F.Mask" "F.Paste")
-			(roundrect_rratio 0.25)
+			(roundrect_rratio 0.217391)
 			(net 2 "+3.3V")
 			(pintype "passive")
 		)
 		(embedded_fonts no)
-		(model "${KICAD9_3DMODEL_DIR}/Capacitor_SMD.3dshapes/C_0603_1608Metric.step"
+		(model "${KICAD9_3DMODEL_DIR}/Capacitor_SMD.3dshapes/C_1206_3216Metric.step"
 			(offset
 				(xyz 0 0 0)
@@
 		)
 	)
-	(footprint "Capacitor_SMD:C_0603_1608Metric"
+	(footprint "Capacitor_SMD:C_1206_3216Metric"
 		(layer "F.Cu")
-		(at 122.12 65.75 180)
-		(descr "Capacitor SMD 0603 (1608 Metric), square (rectangular) end terminal, IPC-7351 nominal, (Body size source: IPC-SM-782 page 76, https://www.pcb-3d.com/wordpress/wp-content/uploads/ipc-sm-782a_amendment_1_and_2.pdf), generated with kicad-footprint-generator")
+		(at 122.12 64 180)
+		(descr "Capacitor SMD 1206 (3216 Metric), square (rectangular) end terminal, IPC-7351 nominal, (Body size source: IPC-SM-782 page 76, https://www.pcb-3d.com/wordpress/wp-content/uploads/ipc-sm-782a_amendment_1_and_2.pdf), generated with kicad-footprint-generator")
 		(tags "capacitor")
 		(property "Reference" "C12"
-			(at 2.97 -0.02 0)
+			(at 0 -1.85 180)
 			(layer "F.SilkS")
+			(hide yes)
 			(effects
 				(font
@@
 		)
 		(property "Value" "22uF"
-			(at 0 1.43 0)
+			(at 0 1.85 180)
 			(layer "F.Fab")
 			(effects
@@
 		)
 		(property "Datasheet" ""
-			(at 0 0 0)
+			(at 0 0 180)
 			(layer "F.Fab")
 			(hide yes)
@@
 		)
 		(property "Description" "Unpolarized capacitor, small symbol"
-			(at 0 0 0)
+			(at 0 0 180)
 			(layer "F.Fab")
 			(hide yes)
@@
 		(attr smd)
 		(fp_line
-			(start -0.14058 0.51)
-			(end 0.14058 0.51)
+			(start -0.711252 0.91)
+			(end 0.711252 0.91)
 			(stroke
 				(width 0.12)
@@
 		)
 		(fp_line
-			(start -0.14058 -0.51)
-			(end 0.14058 -0.51)
+			(start -0.711252 -0.91)
+			(end 0.711252 -0.91)
 			(stroke
 				(width 0.12)
@@
 		)
 		(fp_line
-			(start 1.48 0.73)
-			(end -1.48 0.73)
+			(start 2.3 1.15)
+			(end -2.3 1.15)
 			(stroke
 				(width 0.05)
@@
 		)
 		(fp_line
-			(start 1.48 -0.73)
-			(end 1.48 0.73)
+			(start 2.3 -1.15)
+			(end 2.3 1.15)
 			(stroke
 				(width 0.05)
@@
 		)
 		(fp_line
-			(start -1.48 0.73)
-			(end -1.48 -0.73)
+			(start -2.3 1.15)
+			(end -2.3 -1.15)
 			(stroke
 				(width 0.05)
@@
 		)
 		(fp_line
-			(start -1.48 -0.73)
-			(end 1.48 -0.73)
+			(start -2.3 -1.15)
+			(end 2.3 -1.15)
 			(stroke
 				(width 0.05)
@@
 		)
 		(fp_line
-			(start 0.8 0.4)
-			(end -0.8 0.4)
+			(start 1.6 0.8)
+			(end -1.6 0.8)
 			(stroke
 				(width 0.1)
@@
 		)
 		(fp_line
-			(start 0.8 -0.4)
-			(end 0.8 0.4)
+			(start 1.6 -0.8)
+			(end 1.6 0.8)
 			(stroke
 				(width 0.1)
@@
 		)
 		(fp_line
-			(start -0.8 0.4)
-			(end -0.8 -0.4)
+			(start -1.6 0.8)
+			(end -1.6 -0.8)
 			(stroke
 				(width 0.1)
@@
 		)
 		(fp_line
-			(start -0.8 -0.4)
-			(end 0.8 -0.4)
+			(start -1.6 -0.8)
+			(end 1.6 -0.8)
 			(stroke
 				(width 0.1)
@@
 		)
 		(fp_text user "${REFERENCE}"
-			(at 0 0 0)
+			(at 0 0 180)
 			(layer "F.Fab")
 			(effects
 				(font
-					(size 0.4 0.4)
-					(thickness 0.06)
+					(size 0.8 0.8)
+					(thickness 0.12)
 				)
 			)
 		)
 		(pad "1" smd roundrect
-			(at -0.775 0 180)
-			(size 0.9 0.95)
+			(at -1.475 0 180)
+			(size 1.15 1.8)
 			(layers "F.Cu" "F.Mask" "F.Paste")
-			(roundrect_rratio 0.25)
+			(roundrect_rratio 0.217391)
 			(net 1 "GND")
 			(pintype "passive")
 		)
 		(pad "2" smd roundrect
-			(at 0.775 0 180)
-			(size 0.9 0.95)
+			(at 1.475 0 180)
+			(size 1.15 1.8)
 			(layers "F.Cu" "F.Mask" "F.Paste")
-			(roundrect_rratio 0.25)
+			(roundrect_rratio 0.217391)
 			(net 2 "+3.3V")
 			(pintype "passive")
 		)
 		(embedded_fonts no)
-		(model "${KICAD9_3DMODEL_DIR}/Capacitor_SMD.3dshapes/C_0603_1608Metric.step"
+		(model "${KICAD9_3DMODEL_DIR}/Capacitor_SMD.3dshapes/C_1206_3216Metric.step"
 			(offset
 				(xyz 0 0 0)
@@
 	)
 	(segment
-		(start 123.45 64.11)
-		(end 123.99 63.57)
-		(width 1)
-		(layer "F.Cu")
-		(net 1)
-	)
-	(segment
 		(start 123.74 58.36)
 		(end 123.9 58.52)
@@
 	)
 	(segment
-		(start 122.865 64.695)
-		(end 122.975 64.585)
+		(start 123.565 61.435)
+		(end 124 61)
 		(width 1)
 		(layer "F.Cu")
@@
 	)
 	(segment
-		(start 122.975 64.585)
-		(end 123.45 64.11)
-		(width 1)
-		(layer "F.Cu")
-		(net 1)
-	)
-	(segment
 		(start 151.7 99.715)
 		(end 151.7 100.38)
@@
 	)
 	(segment
+		(start 123.565 66.89)
+		(end 123.565 61.435)
+		(width 1)
+		(layer "F.Cu")
+		(net 1)
+	)
+	(segment
 		(start 147.83 98.845)
 		(end 148.025 99.04)
@@
 		(net 1)
 	)
-	(segment
-		(start 122.865 67.64)
-		(end 122.865 64.695)
-		(width 1)
-		(layer "F.Cu")
-		(net 1)
-	)
 	(via
 		(at 101.6 121.92)
@@
 	)
 	(via
-		(at 142.24 121.92)
+		(at 124 61)
 		(size 0.6)
 		(drill 0.3)
 		(layers "F.Cu" "B.Cu")
-		(free yes)
 		(net 1)
 	)
 	(via
-		(at 123.99 63.57)
+		(at 142.24 121.92)
 		(size 0.6)
 		(drill 0.3)
 		(layers "F.Cu" "B.Cu")
+		(free yes)
 		(net 1)
 	)
@@
 		(polygon
 			(pts
-				(xy 122.69 76.3) (xy 122.67 68.75) (xy 122.09 67.64) (xy 122.12 65.75) (xy 122.12 64.73) (xy 120.52 64.73)
-				(xy 118.66 64.7) (xy 118.69 76.28)
+				(xy 122.69 76.3) (xy 122.67 68.75) (xy 122.09 67.64) (xy 122.12 65.75) (xy 122.12 63) (xy 120.52 63)
+				(xy 118.66 63) (xy 118.69 76.28)
 			)
 		)
